File: pcb/PCB Main/External Connections.kicad_sch (KiCad schematic)
At the start: 14 parts, among them CN1 Conn_01x07, CN2 Conn_01x02, CN3 Conn_01x02, CN4 Conn_01x04, CN5 Conn_01x04, CN6 Conn_01x03, CN7 Conn_01x03, CN8 Conn_01x03, CN9 Conn_01x02

Commit message: retoques
Changed lines of the file:
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@@
 		)
 	)
-	(text_box "Pin 1 (Vref) doesn't supply the STM32, it's just voltage reference for STLINK. Pin 19 does."
+	(text_box "Pin 1 (Vref) doesn't supply the STM32, it's just voltage reference for STLINK. Pin 7 does."
 		(exclude_from_sim no)
 		(at 210.82 102.87 0)

Commit message: silkscreen
Parts:
- BT1: footprint PZG_Batteries:SMTU2032C -> PZG_Batteries:1066; Component SMTU2032-C -> 1066; Manufacturer Renata -> KEYSTONE; Package SMD -> PTH; Supplier Mouser -> Farnell; Supplier Part # 614-SMTU2032-C -> 1339839
Changed lines of the file:
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@@
 		(dnp no)
 		(property "Reference" "BT1"
-			(at 189.23 57.15 0)
+			(at 187.96 57.15 0)
 			(effects
 				(font
@@
 		)
 		(property "Value" "CR2032"
-			(at 184.15 59.69 0)
+			(at 186.69 59.69 0)
 			(effects
 				(font
@@
 			)
 		)
-		(property "Footprint" "PZG_Batteries:SMTU2032C"
+		(property "Footprint" "PZG_Batteries:1066"
 			(at 196.85 158.42 0)
 			(effects
@@
 			)
 		)
-		(property "Component" "SMTU2032-C"
+		(property "Component" "1066"
 			(at 180.34 63.5 0)
 			(effects
@@
 			)
 		)
-		(property "Manufacturer" "Renata"
+		(property "Manufacturer" "KEYSTONE"
 			(at 180.34 63.5 0)
 			(effects
@@
 			)
 		)
-		(property "Package" "SMD"
+		(property "Package" "PTH"
 			(at 180.34 63.5 0)
 			(effects
@@
 			)
 		)
-		(property "Supplier" "Mouser"
+		(property "Supplier" "Farnell"
 			(at 180.34 63.5 0)
 			(effects
@@
 			)
 		)
-		(property "Supplier Part #" "614-SMTU2032-C"
+		(property "Supplier Part #" "1339839"
 			(at 180.34 63.5 0)
 			(effects

Commit message: pcb sent to jlcpcb
Parts:
- BT1: now left out of the parts list
- CN1: Package (none) -> PTH; Supplier Part Type (none) -> -; now left out of the parts list
- CN2, CN3: Manufacturer (none) -> JST; Package (none) -> PTH; now left out of the parts list
- CN4, CN5, CN6, CN7, CN8, CN9: Package (none) -> PTH; now left out of the parts list
Connections:
- net DFR0198: now also CN6.1 (Pin_1); no longer CN6.2 (Pin_2)
- net GND: now also CN6.2 (Pin_2); no longer CN6.3 (Pin_3)
- net SEN0308: now also CN7.1 (Pin_1); no longer CN7.2 (Pin_2)
- net VDD_SENS: now also CN6.3 (Pin_3), CN7.2 (Pin_2); no longer CN6.1 (Pin_1), CN7.1 (Pin_1)
Other:
- note added: "USART"
- note removed: "UART"
Changed lines of the file:
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@@
 		)
 	)
-	(text "UART"
+	(text "USART"
 		(exclude_from_sim no)
 		(at 48.26 125.73 0)
@@
 	(wire
 		(pts
-			(xy 180.34 105.41) (xy 185.42 105.41)
+			(xy 180.34 105.41) (xy 186.69 105.41)
 		)
 		(stroke
@@
 	(wire
 		(pts
-			(xy 140.97 105.41) (xy 146.05 105.41)
+			(xy 140.97 105.41) (xy 147.32 105.41)
 		)
 		(stroke
@@
 	(wire
 		(pts
-			(xy 146.05 110.49) (xy 146.05 111.76)
-		)
-		(stroke
-			(width 0)
-			(type default)
-		)
-	)
-	(wire
-		(pts
 			(xy 62.23 111.76) (xy 67.31 111.76)
 		)
@@
 	(wire
 		(pts
-			(xy 180.34 107.95) (xy 186.69 107.95)
+			(xy 180.34 107.95) (xy 185.42 107.95)
 		)
 		(stroke
@@
 		)
 	)
-	(global_label "DFR0198"
-		(shape output)
-		(at 147.32 107.95 0)
-		(fields_autoplaced yes)
-		(effects
-			(font
-				(size 1.27 1.27)
-			)
-			(justify left)
-		)
-		(property "Intersheetrefs" "${INTERSHEET_REFS}"
-			(at 158.7718 107.95 0)
-			(effects
-				(font
-					(size 1.27 1.27)
-				)
-				(justify left)
-				(hide yes)
-			)
-		)
-	)
-	(global_label "SEN0308"
-		(shape output)
-		(at 186.69 107.95 0)
-		(fields_autoplaced yes)
-		(effects
-			(font
-				(size 1.27 1.27)
-			)
-			(justify left)
-		)
-		(property "Intersheetrefs" "${INTERSHEET_REFS}"
-			(at 198.2022 107.95 0)
-			(effects
-				(font
-					(size 1.27 1.27)
-				)
-				(justify left)
-				(hide yes)
-			)
-		)
-	)
 	(global_label "VDD_SENS"
 		(shape input)
-		(at 185.42 105.41 0)
+		(at 146.05 110.49 0)
 		(fields_autoplaced yes)
 		(effects
@@
 		)
 		(property "Intersheetrefs" "${INTERSHEET_REFS}"
-			(at 197.8999 105.41 0)
+			(at 158.5299 110.49 0)
 			(effects
 				(font
@@
 	(global_label "VDD_SENS"
 		(shape input)
-		(at 146.05 105.41 0)
+		(at 67.31 104.14 0)
 		(fields_autoplaced yes)
 		(effects
@@
 		)
 		(property "Intersheetrefs" "${INTERSHEET_REFS}"
-			(at 158.5299 105.41 0)
+			(at 79.7899 104.14 0)
 			(effects
 				(font
@@
 	(global_label "VDD_SENS"
 		(shape input)
-		(at 67.31 104.14 0)
+		(at 106.68 104.14 0)
 		(fields_autoplaced yes)
 		(effects
@@
 		)
 		(property "Intersheetrefs" "${INTERSHEET_REFS}"
-			(at 79.7899 104.14 0)
+			(at 119.1599 104.14 0)
 			(effects
 				(font
@@
 		)
 	)
-	(global_label "VDD_SENS"
-		(shape input)
-		(at 106.68 104.14 0)
+	(global_label "DFR0198"
+		(shape output)
+		(at 147.32 105.41 0)
 		(fields_autoplaced yes)
 		(effects
@@
 		)
 		(property "Intersheetrefs" "${INTERSHEET_REFS}"
-			(at 119.1599 104.14 0)
+			(at 158.7718 105.41 0)
 			(effects
 				(font
@@
 		)
 	)
+	(global_label "SEN0308"
+		(shape output)
+		(at 186.69 105.41 0)
+		(fields_autoplaced yes)
+		(effects
+			(font
+				(size 1.27 1.27)
+			)
+			(justify left)
+		)
+		(property "Intersheetrefs" "${INTERSHEET_REFS}"
+			(at 198.2022 105.41 0)
+			(effects
+				(font
+					(size 1.27 1.27)
+				)
+				(justify left)
+				(hide yes)
+			)
+		)
+	)
 	(global_label "SWCLK"
 		(shape output)
@@
 		)
 	)
+	(global_label "VDD_SENS"
+		(shape input)
+		(at 185.42 107.95 0)
+		(fields_autoplaced yes)
+		(effects
+			(font
+				(size 1.27 1.27)
+			)
+			(justify left)
+		)
+		(property "Intersheetrefs" "${INTERSHEET_REFS}"
+			(at 197.8999 107.95 0)
+			(effects
+				(font
+					(size 1.27 1.27)
+				)
+				(justify left)
+				(hide yes)
+			)
+		)
+	)
 	(global_label "SDA"
 		(shape bidirectional)
@@
 		(unit 1)
 		(exclude_from_sim no)
-		(in_bom yes)
+		(in_bom no)
 		(on_board yes)
 		(dnp no)
@@
 			)
 		)
+		(property "Package" "PTH"
+			(at 57.15 138.43 0)
+			(effects
+				(font
+					(size 1.27 1.27)
+				)
+				(hide yes)
+			)
+		)
 		(pin "2"
 		)
@@
 		(unit 1)
 		(exclude_from_sim no)
-		(in_bom yes)
+		(in_bom no)
 		(on_board yes)
 		(dnp no)
@@
 		(unit 1)
 		(exclude_from_sim no)
-		(in_bom yes)
+		(in_bom no)
 		(on_board yes)
 		(dnp no)
@@
 			)
 		)
+		(property "Package" "PTH"
+			(at 57.15 106.68 0)
+			(effects
+				(font
+					(size 1.27 1.27)
+				)
+				(hide yes)
+			)
+		)
 		(pin "2"
 		)
@@
 		(unit 1)
 		(exclude_from_sim no)
-		(in_bom yes)
+		(in_bom no)
 		(on_board yes)
 		(dnp no)
@@
 			)
 		)
+		(property "Package" "PTH"
+			(at 175.26 107.95 0)
+			(effects
+				(font
+					(size 1.27 1.27)
+				)
+				(hide yes)
+			)
+		)
 		(pin "2"
 		)
@@
 		(unit 1)
 		(exclude_from_sim no)
-		(in_bom yes)
+		(in_bom no)
 		(on_board yes)
 		(dnp no)
@@
 			)
 		)
+		(property "Package" "PTH"
+			(at 96.52 106.68 0)
+			(effects
+				(font
+					(size 1.27 1.27)
+				)
+				(hide yes)
+			)
+		)
 		(pin "2"
 		)
@@
 		(unit 1)
 		(exclude_from_sim no)
-		(in_bom yes)
+		(in_bom no)
 		(on_board yes)
 		(dnp no)
@@
 			)
 		)
+		(property "Package" "PTH"
+			(at 135.89 107.95 0)
+			(effects
+				(font
+					(size 1.27 1.27)
+				)
+				(hide yes)
+			)
+		)
 		(pin "2"
 		)
@@
 		(unit 1)
 		(exclude_from_sim no)
-		(in_bom yes)
+		(in_bom no)
 		(on_board yes)
 		(dnp no)
@@
 			)
 		)
+		(property "Package" "PTH"
+			(at 95.25 135.89 0)
+			(effects
+				(font
+					(size 1.27 1.27)
+				)
+				(hide yes)
+			)
+		)
 		(pin "1"
 		)
@@
 		(unit 1)
 		(exclude_from_sim no)
-		(in_bom yes)
+		(in_bom no)
 		(on_board yes)
 		(dnp no)
@@
 			)
 		)
-		(property "Description" ""
+		(property "Description" "01x02 2.5mm Pin Connector Horizontal"
 			(at 81.28 74.93 0)
 			(effects
@@
 			)
 		)
+		(property "Package" "PTH"
+			(at 81.28 74.93 0)
+			(effects
+				(font
+					(size 1.27 1.27)
+				)
+				(hide yes)
+			)
+		)
+		(property "Manufacturer" "JST"
+			(at 81.28 74.93 0)
+			(effects
+				(font
+					(size 1.27 1.27)
+				)
+				(hide yes)
+			)
+		)
 		(pin "1"
 		)
@@
 		(unit 1)
 		(exclude_from_sim no)
-		(in_bom yes)
+		(in_bom no)
 		(on_board yes)
 		(dnp no)
@@
 			)
 		)
-		(property "Description" "Generic connector, single row, 01x07, script generated (kicad-library-utils/schlib/autogen/connector/)"
+		(property "Description" "01x07 2.54mm Pin Header Vertical"
+			(at 231.14 71.12 0)
+			(effects
+				(font
+					(size 1.27 1.27)
+				)
+				(hide yes)
+			)
+		)
+		(property "Package" "PTH"
+			(at 231.14 71.12 0)
+			(effects
+				(font
+					(size 1.27 1.27)
+				)
+				(hide yes)
+			)
+		)
+		(property "Supplier Part Type" "-"
 			(at 231.14 71.12 0)
 			(effects
@@
 	(symbol
 		(lib_id "power:GND")
-		(at 146.05 111.76 0)
+		(at 147.32 107.95 90)
 		(unit 1)
 		(exclude_from_sim no)
@@
 		(fields_autoplaced yes)
 		(property "Reference" "#PWR063"
-			(at 146.05 118.11 0)
+			(at 153.67 107.95 0)
 			(effects
 				(font
@@
 		)
 		(property "Value" "GND"
-			(at 146.05 116.84 0)
+			(at 151.13 107.9499 90)
 			(effects
 				(font
 					(size 1.27 1.27)
 				)
+				(justify right)
 			)
 		)
 		(property "Footprint" ""
-			(at 146.05 111.76 0)
+			(at 147.32 107.95 0)
 			(effects
 				(font
@@
 		)
 		(property "Datasheet" ""
-			(at 146.05 111.76 0)
+			(at 147.32 107.95 0)
 			(effects
 				(font
@@
 		)
 		(property "Description" "Power symbol creates a global label with name \"GND\" , ground"
-			(at 146.05 111.76 0)
+			(at 147.32 107.95 0)
 			(effects
 				(font
@@
 		(unit 1)
 		(exclude_from_sim no)
-		(in_bom yes)
+		(in_bom no)
 		(on_board yes)
 		(dnp no)
@@
 			)
 		)
-		(property "Description" ""
+		(property "Description" "01x02 2.5mm Pin Connector Horizontal"
 			(at 124.46 74.93 0)
 			(effects
@@
 			(at 124.46 74.93 0)
 			(effects
+				(font
+					(size 1.27 1.27)
+				)
+				(hide yes)
+			)
+		)
+		(property "Package" "PTH"
+			(at 124.46 74.93 0)
+			(effects
+				(font
+					(size 1.27 1.27)
+				)
+				(hide yes)
+			)
+		)
+		(property "Manufacturer" "JST"
+			(at 124.46 74.93 0)
+			(effects
