File: pcb/PCB Main/PCB Main.kicad_pcb (KiCad board)
At the start: 2 copper layers, 35 parts, among them CN1 Conn_ARM_JTAG_SWD_10, J1 Conn_01x03, J2 Conn_01x02, J3 Conn_01x02, J4 Conn_01x02, U1 STM32WB55RGVx, U2 AEM10941, U3 INA3221, Y1 32MHz, Y2 32.768kHz

Commit message: updates
Parts:
- added SW1: SW_Push, Button_Switch_SMD:SW_SPST_TL3342, F.Cu at (87.4, 44.2)
- moved CN1 5.39 mm to (113.3, 45.1), turned to -90 degrees
- renumbered D2 to LED1, D3 to LED2
Connections:
- net VBAT renamed VBATT
- U1 pad 17: unconnected-(U1-PA2-Pad17) -> /STM32WB55RG/DFR0198
- U1 pad 23: unconnected-(U1-PA8-Pad23) -> /STM32WB55RG/SEN0308
- U1 pad 24: /STM32WB55RG/USART_RX -> unconnected-(U1-PA9-Pad24)
- U1 pad 31: unconnected-(U1-RF1-Pad31) -> RF1
- U1 pad 51: /STM32WB55RG/USART_TX -> unconnected-(U1-PA10-Pad51)
- U1 pad 66: unconnected-(U1-PB6-Pad66) -> /STM32WB55RG/USART_RX
- U1 pad 67: unconnected-(U1-PB7-Pad67) -> /STM32WB55RG/USART_TX

Commit message: PCB casi lista
Parts:
- removed J2: Conn_01x02, Connector_PinHeader_2.54mm:PinHeader_1x02_P2.54mm_Vertical
- removed J3, J4: Conn_01x02, Connector_PinHeader_1.27mm:PinHeader_1x02_P1.27mm_Vertical
- added BT1: CR2032, PZG_Batteries:SMTU2032C, B.Cu at (38.5, 52.6)
- added C11: 100nF, Capacitor_SMD:C_0402_1005Metric, F.Cu at (46.5, 63.0)
- added C12: 100nF, Capacitor_SMD:C_0402_1005Metric, F.Cu at (44.7, 46.9)
- added C13: 100nF, Capacitor_SMD:C_0402_1005Metric, F.Cu at (35.3, 43.8)
- added C14: 100nF, Capacitor_SMD:C_0402_1005Metric, F.Cu at (41.7, 35.8)
- added C15: 4.7uF, Capacitor_SMD:C_0402_1005Metric, F.Cu at (34.0, 42.4)
- added C16: 100nF, Capacitor_SMD:C_0402_1005Metric, F.Cu at (35.1, 41.4)
- added C17: 100nF, Capacitor_SMD:C_0402_1005Metric, F.Cu at (48.5, 38.6)
- added C18: 100nF, Capacitor_SMD:C_0402_1005Metric, F.Cu at (39.6, 47.0)
- added C19: 100nF, Capacitor_SMD:C_0402_1005Metric, F.Cu at (37.3, 34.5)
- added C20: 100pF, Capacitor_SMD:C_0402_1005Metric, F.Cu at (37.3, 35.6)
- added C21: 100nF, Capacitor_SMD:C_0402_1005Metric, F.Cu at (45.7, 46.7)
- added C22: 4.7uF, Capacitor_SMD:C_0402_1005Metric, F.Cu at (35.1, 38.9)
- added C23: 100nF, Capacitor_SMD:C_0402_1005Metric, F.Cu at (51.1, 41.1)
- added C24: 15pF, Capacitor_SMD:C_0402_1005Metric, F.Cu at (48.8, 45.1)
- added C25: 15pF, Capacitor_SMD:C_0402_1005Metric, F.Cu at (48.8, 41.0)
- added C26: 100nF, Capacitor_SMD:C_0402_1005Metric, F.Cu at (49.9, 48.4)
- added C27: 100nF, Capacitor_SMD:C_0402_1005Metric, F.Cu at (74.2, 26.4)
- added C28: 100nF, Capacitor_SMD:C_0402_1005Metric, F.Cu at (64.1, 26.4)
- added C29: 1.2pF, Capacitor_SMD:C_0402_1005Metric, F.Cu at (39.1, 22.7)
- added CN2: Conn_01x02, Connector_JST:JST_EH_S2B-EH_1x02_P2.50mm_Horizontal, F.Cu at (72.8, 23.9)
- added CN3: Conn_01x02, Connector_JST:JST_EH_S2B-EH_1x02_P2.50mm_Horizontal, F.Cu at (63.1, 23.9)
- added CN4: Conn_01x04, Connector_PinHeader_2.54mm:PinHeader_1x04_P2.54mm_Horizontal, F.Cu at (81.2, 38.7)
- added CN5: Conn_01x04, Connector_PinHeader_2.54mm:PinHeader_1x04_P2.54mm_Horizontal, F.Cu at (81.2, 51.4)
- added CN6: Conn_01x03, Connector_PinHeader_2.54mm:PinHeader_1x03_P2.54mm_Horizontal, F.Cu at (78.6, 66.5)
- added CN7: Conn_01x03, Connector_PinHeader_2.54mm:PinHeader_1x03_P2.54mm_Horizontal, F.Cu at (69.2, 66.5)
- added CN8: Conn_01x03, Connector_PinHeader_2.54mm:PinHeader_1x03_P2.54mm_Vertical, F.Cu at (60.3, 67.9)
- added CN9: Conn_01x02, Connector_PinHeader_2.54mm:PinHeader_1x02_P2.54mm_Vertical, F.Cu at (56.1, 65.4)
- added FLT1: Low_Pass_Filter_2.4GHz_50R, MLPF-WB55-01E3:MLPF-WB55-01E3, F.Cu at (39.9, 34.8)
- added H1: MountingHole, MountingHole:MountingHole_2.2mm_M2, F.Cu at (23.6, 24.1)
- added H2: MountingHole, MountingHole:MountingHole_2.2mm_M2, F.Cu at (82.9, 24.1)
- added H3: MountingHole, MountingHole:MountingHole_2.2mm_M2, F.Cu at (82.9, 68.1)
- added H4: MountingHole, MountingHole:MountingHole_2.2mm_M2, F.Cu at (23.6, 68.1)
- added L4: 10nH, Inductor_SMD:L_0402_1005Metric, F.Cu at (35.1, 40.4)
- added L5: 10uH, Inductor_SMD:L_0805_2012Metric, F.Cu at (32.5, 39.6)
- added L6: 3.6nH, LED_SMD:LED_0402_1005Metric, F.Cu at (39.6, 24.5)
- added Q1: AO3401A, Package_TO_SOT_SMD:SOT-23, F.Cu at (59.1, 27.7)
- added R10: 10k, Resistor_SMD:R_0402_1005Metric, F.Cu at (70.6, 39.1)
- added R11: 10k, Resistor_SMD:R_0402_1005Metric, F.Cu at (50.4, 35.1)
- added R12: 10k, Resistor_SMD:R_0402_1005Metric, F.Cu at (48.8, 34.3)
- added R13: 10k, Resistor_SMD:R_0402_1005Metric, F.Cu at (48.5, 46.5)
- added R14: 10k, Resistor_SMD:R_0402_1005Metric, F.Cu at (53.1, 39.6)
- added R15: 10k, Resistor_SMD:R_0402_1005Metric, F.Cu at (51.8, 38.4)
- added R16: 470, Resistor_SMD:R_0402_1005Metric, F.Cu at (28.4, 34.0)
- added R17: 300, Resistor_SMD:R_0402_1005Metric, F.Cu at (28.4, 36.6)
- added R18: 100k, Resistor_SMD:R_0402_1005Metric, F.Cu at (56.5, 27.7)
- added R19: 10k, Resistor_SMD:R_0402_1005Metric, F.Cu at (42.8, 55.8)
- added U4: MB85RS256B, Package_SO:SOIC-8_3.9x4.9mm_P1.27mm, F.Cu at (38.3, 56.9)
- C1: value 0.1uF -> 100nF; footprint Capacitor_SMD:C_0603_1608Metric -> Capacitor_SMD:C_0402_1005Metric
- C10: value 10uF -> 100nF; footprint Capacitor_SMD:C_0805_2012Metric -> Capacitor_SMD:C_0402_1005Metric
- C2, C3, C4: value 33nF -> 100nF; footprint Capacitor_SMD:C_0603_1608Metric -> Capacitor_SMD:C_0402_1005Metric
- C5, C6, C7, C8: footprint Capacitor_SMD:C_0805_2012Metric -> Capacitor_SMD:C_0603_1608Metric
- C9: value 220uF -> 150uF; footprint Capacitor_SMD:CP_Elec_8x6.2 -> Capacitor_SMD:C_1206_3216Metric
- CN1: value Conn_ARM_JTAG_SWD_10 -> Conn_01x07; footprint Connector_PinHeader_1.27mm:PinHeader_2x05_P1.27mm_Vertical -> Connector_PinHeader_2.54mm:PinHeader_1x07_P2.54mm_Vertical
- D1: value BAT54J -> D_Schottky; footprint Diode_SMD:D_SOD-323F -> Diode_SMD:D_SOD-323
- L2: footprint Inductor_SMD:L_0805_2012Metric -> Inductor_SMD:L_0603_1608Metric
- L3: value 600 -> 600@100MHz
- LED1: value GREEN -> Green; footprint LED_SMD:LED_0603_1608Metric -> LED_SMD:LED_0805_2012Metric
- LED2: value BLUE -> White; footprint LED_SMD:LED_0603_1608Metric -> LED_SMD:LED_0805_2012Metric
- R1, R2, R3: value 0.1 -> 0.33
- R4, R5, R6, R7, R8, R9: footprint Resistor_SMD:R_0603_1608Metric -> Resistor_SMD:R_0402_1005Metric
- SW1: value SW_Push -> SW_Reset
- moved X1 89.8 mm to (34.8, 36.6)
- moved LED1 84.5 mm to (25.7, 34.0)
- moved LED2 84.4 mm to (25.7, 36.6)
- moved CN1 84.2 mm to (31.6, 65.4), turned to 90 degrees
- moved X2 76.6 mm to (48.3, 43.1), turned to 90 degrees
- moved SW1 61.5 mm to (25.9, 45.6), turned to 90 degrees
- moved D1 58.1 mm to (52.6, 42.0), turned to 90 degrees
- moved R1 57.5 mm to (74.7, 35.1), turned to -90 degrees
- moved R4 53.5 mm to (72.1, 34.0), turned to 90 degrees
- moved C5 53.2 mm to (65.0, 61.5), turned to -90 degrees
- moved R5 50.7 mm to (72.1, 36.1), turned to -90 degrees
- moved L1 50.4 mm to (68.3, 59.9), turned to -90 degrees
- moved C2 49.3 mm to (71.1, 35.1), turned to 90 degrees
- moved C7 45.7 mm to (69.8, 56.6), turned to 0 degrees
- moved C1 43.4 mm to (64.1, 37.1), turned to -90 degrees
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- renumbered Y1 to X1, Y2 to X2
Connections:
- net /Power Management/BAT+ renamed VBAT
- net /Power Management/PV+ renamed VSRC
- net /STM32WB55RG/OSC32_IN renamed /STM32WB55RG/LSE_IN
- net /STM32WB55RG/OSC32_OUT renamed /STM32WB55RG/LSE_OUT
- net /STM32WB55RG/OSC_IN renamed /STM32WB55RG/HSE_IN
- net /STM32WB55RG/OSC_OUT renamed /STM32WB55RG/HSE_OUT
- net /STM32WB55RG/SWCLK renamed SWCLK
- net S0 renamed S0_AEM
- net S1 renamed S1_AEM
- net S2 renamed S2_AEM
- C10 pad 1: /Power Management/BATT -> +3.3V
- C9 pad 1: GND -> /Power Management/BATT
- C9 pad 2: /Power Management/BATT -> GND
- CN1 pad 2: /STM32WB55RG/SWDIO -> NRST
- CN1 pad 3: GND -> SWO
- CN1 pad 5: GND -> SWDIO
- CN1 pad 6: /STM32WB55RG/SWO -> GND
- CN1 pad 7: unconnected-(CN1-KEY-Pad7) -> 3V3_EXT
- D1 pad 1: /STM32WB55RG/NRST -> NRST
- J1 pad 1: /Power Management/3V3_EXT -> 3V3_EXT
- J1 pad 2: +3.3V -> /Power Management/3V3
- L1 pad 1: Net-(U2-BUFSRC) -> Net-(U2-SWBOOST)
- L1 pad 2: Net-(U2-SWBOOST) -> Net-(U2-BUFSRC)
- LED2 pad 1: /STM32WB55RG/USER_LED -> GND
- R3 pad 1: /Power Management/HVOUT -> /Power Management/3V3
- R3 pad 2: /Power Management/3V3 -> +3.3V
- R8 pad 2: /Power Management/HVOUT -> /Power Management/3V3
- R9 pad 2: /Power Management/3V3 -> +3.3V
- SW1 pad 2: /STM32WB55RG/NRST -> NRST
- U1 pad 1: VBATT -> VBAT_BACKUP
- U1 pad 10: unconnected-(U1-PC1-Pad10) -> SDA
- U1 pad 11: unconnected-(U1-PC2-Pad11) -> GATE_SENS
- U1 pad 15: unconnected-(U1-PA0-Pad15) -> PV_INA
- U1 pad 16: unconnected-(U1-PA1-Pad16) -> CRI_INA
- U1 pad 17: /STM32WB55RG/DFR0198 -> WAR_INA
- U1 pad 22: unconnected-(U1-PA7-Pad22) -> DFR0198
- U1 pad 23: /STM32WB55RG/SEN0308 -> SEN0308
- U1 pad 47: unconnected-(U1-PB13-Pad47) -> SCK
- U1 pad 48: unconnected-(U1-PB14-Pad48) -> MISO
- U1 pad 49: unconnected-(U1-PB15-Pad49) -> MOSI
- U1 pad 51: unconnected-(U1-PA10-Pad51) -> /STM32WB55RG/USER_LED
- U1 pad 52: unconnected-(U1-PA11-Pad52) -> CS_FRAM
- U1 pad 54: /STM32WB55RG/SWDIO -> SWDIO
- U1 pad 6: SCL -> unconnected-(U1-PB8-Pad6)
- U1 pad 60: unconnected-(U1-PC12-Pad60) -> WP_FRAM
- U1 pad 63: /STM32WB55RG/SWO -> SWO
- U1 pad 65: /STM32WB55RG/USER_LED -> unconnected-(U1-PB5-Pad65)
- U1 pad 66: /STM32WB55RG/USART_RX -> USART_RX
- U1 pad 67: /STM32WB55RG/USART_TX -> USART_TX
- U1 pad 7: SDA -> unconnected-(U1-PB9-Pad7)
- U1 pad 9: unconnected-(U1-PC0-Pad9) -> SCL
- U2 pad 26: unconnected-(U2-FB_COLD-Pad26) -> /Power Management/SRC
- U3 pad 10: unconnected-(U3-PV-Pad10) -> PV_INA
- U3 pad 16: unconnected-(U3-VPU-Pad16) -> +3.3V
- U3 pad 8: unconnected-(U3-WARNING-Pad8) -> WAR_INA
- U3 pad 9: unconnected-(U3-CRITICAL-Pad9) -> CRI_INA
Routing:
- net +3.3V: track 0.00 -> 176.3 mm, vias 0 -> 16
- net VDD_SENS: track 0.00 -> 72.9 mm, vias 0 -> 1
- net /Power Management/BATT: track 0.00 -> 60.2 mm, vias 0 -> 2
- net NRST: track 0.00 -> 57.8 mm, vias 0 -> 2
- net SCL: track 0.00 -> 57.5 mm, vias 0 -> 2
- net SDA: track 0.00 -> 55.7 mm, vias 0 -> 1
- net DFR0198: track 0.00 -> 53.9 mm, vias 0 -> 1
- net SEN0308: track 0.00 -> 45.3 mm, vias 0 -> 1
- net PV_INA: track 0.00 -> 37.9 mm, vias 0 -> 2
- net S2_AEM: track 0.00 -> 36.3 mm, vias 0 -> 2
- net S1_AEM: track 0.00 -> 35.7 mm, vias 0 -> 2
- net CRI_INA: track 0.00 -> 34.8 mm, vias 0 -> 2
- net S0_AEM: track 0.00 -> 34.8 mm, vias 0 -> 2
- net WAR_INA: track 0.00 -> 33.7 mm, vias 0 -> 2
- net GND: track 0.00 -> 32.9 mm, vias 0 -> 46
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- added copper zone on F.Cu, net /Power Management/BATT
- added copper zone on F.Cu, net /Power Management/BUCK
- added copper zone on F.Cu, net /Power Management/SRC
- added copper zone on B.Cu, net GND
- added copper zone on F.Cu, net GND
- added copper zone on In1.Cu, net GND
- added copper zone on In2.Cu, net GND
Other:
- board outline added: 64.1 x 53 mm
- copper layers 2 -> 4

Commit message: RF hecho
Parts:
- moved CN9 2.29 mm to (53.8, 65.4)
- moved CN8 1.65 mm to (58.7, 67.9)
- moved C15 0.51 mm to (34.5, 42.4)
- moved C12 0.35 mm to (44.7, 47.2)
- moved C16 0.25 mm to (34.8, 41.4)
- moved C18 0.13 mm to (39.6, 47.1)
- moved FLT1 0.08 mm to (40.0, 34.8)
Routing:
- net +3.3V: track 176.3 -> 46.2 mm, vias 16 -> 18
- net VDD_SENS: track 72.9 -> 1.10 mm
- net /Power Management/BATT: track 60.2 -> 4.62 mm
- net /RF/ANT: track 0.00 -> 44.1 mm
- net 3V3_EXT: track 27.1 -> 0.92 mm
- net /Power Management/SRC: track 28.6 -> 4.36 mm
- net Net-(FLT1-PadOUT): track 0.00 -> 9.21 mm
- net /Power Management/3V3: track 11.4 -> 4.49 mm
- net /Power Management/HVOUT: track 8.13 -> 2.36 mm, vias 0 -> 1
- net USART_TX: track 29.9 -> 28.3 mm
- net USART_RX: track 32.9 -> 31.4 mm
- net S2_AEM: track 36.3 -> 37.3 mm
- net S0_AEM: track 34.8 -> 35.6 mm
- net S1_AEM: track 35.7 -> 36.4 mm
- net PV_INA: track 37.9 -> 37.1 mm
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- added copper zone on In2.Cu, net +3.3V
- added copper zone on In2.Cu, net /Power Management/3V3
- added copper zone on In2.Cu, net /Power Management/BATT
- added copper zone on In2.Cu, net /Power Management/HVOUT
- added copper zone on In2.Cu, net /Power Management/SRC
- added copper zone on In2.Cu, net 3V3_EXT
- added copper zone on In2.Cu, net VDD_SENS
Other:
- board size 64.1 x 53 mm -> 64.1 x 56.5 mm

Commit message: retoques
Parts:
- moved C26 0.88 mm to (50.4, 49.1)
- moved C9 0.38 mm to (59.8, 51.6)
Routing:
- net /Power Management/BATT: track 4.62 -> 7.24 mm
- removed copper zone on F.Cu, net /Power Management/BATT

Commit message: vias pad GND
Parts:
- added C29: 1.2pF, Capacitor_SMD:C_0402_1005Metric, F.Cu at (39.2, 26.2)
- C24, C25: value 15pF -> 12pF
- R1, R2, R3: value 0.33 -> 0.22
- renumbered C29 to C30
Routing:
- net GND: track 33.5 -> 40.1 mm, vias 74 -> 134
- net +3.3V: track 46.2 -> 47.0 mm

Commit message: islas cristales
Parts:
- moved D1 15.4 mm to (41.0, 52.2)
- moved C23 15.1 mm to (39.5, 50.8)
- moved X1 7.62 mm to (27.2, 36.1)
- moved R13 6.72 mm to (41.9, 47.8)
- moved C18 6.35 mm to (33.3, 47.5)
- moved C2 6.35 mm to (64.8, 35.5)
- moved CN4 6.35 mm to (74.8, 39.1)
- moved CN6 6.35 mm to (72.2, 66.9)
- moved CN7 6.35 mm to (62.9, 66.9)
- moved FLT1 6.35 mm to (33.6, 35.2)
- moved H3 6.35 mm to (76.6, 68.5)
- moved R1 6.35 mm to (68.3, 35.5)
- moved BT1 6.35 mm to (32.1, 53.0)
- moved C1 6.35 mm to (57.8, 37.5)
- moved C12 6.35 mm to (38.4, 47.7)
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Connections:
- U1 pad 11: GATE_SENS -> unconnected-(U1-PC2-Pad11)
- U1 pad 21: unconnected-(U1-PA6-Pad21) -> GATE_SENS
Routing:
- net /RF/ANT: track 44.1 -> 2.42 mm
- net GND: track 40.1 -> 68.7 mm, vias 134 -> 164
- net NRST: track 57.8 -> 45.9 mm
- net GATE_SENS: track 29.1 -> 20.7 mm, vias 2 -> 0
- net Net-(D1-A): track 7.66 -> 15.8 mm, vias 0 -> 2
- net /STM32WB55RG/BOOT0: track 6.47 -> 10.8 mm
- net DFR0198: track 53.9 -> 55.7 mm
- net SEN0308: track 45.3 -> 47.0 mm
- net /STM32WB55RG/HSE_OUT: track 3.36 -> 5.00 mm
- net /STM32WB55RG/HSE_IN: track 4.24 -> 5.55 mm
- net +3.3V: track 47.0 -> 46.0 mm
- net PV_INA: track 37.1 -> 37.8 mm
- net CRI_INA: track 34.8 -> 35.3 mm
- net WAR_INA: track 33.7 -> 34.2 mm
- net VBAT_BACKUP: track 13.1 -> 13.7 mm
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- added copper zone on F.Cu, net /RF/ANT
Other:
- board text added: "islas cristales - OK plano 3.3V aislado de antena - OK vias debajo pads GND micros - OK antena como zona, no pista - OK cambiar pila holder optimizar pistas poner comentarios silkscreen"

Commit message: silkscreen
Parts:
- BT1: footprint PZG_Batteries:SMTU2032C -> PZG_Batteries:1066
- moved BT1 8.74 mm to (39.4, 57.9)
- moved C26 6.35 mm to (43.0, 55.8), turned to 90 degrees
- moved CN6 2.07 mm to (72.1, 69.0)
- moved CN7 2.03 mm to (62.9, 68.9)
- moved CN9 1.93 mm to (45.6, 66.0)
- moved H3 1.69 mm to (76.6, 70.2)
- moved H4 1.69 mm to (17.3, 70.2)
- moved C30 1.01 mm to (32.8, 22.1)
- moved L6 1.01 mm to (33.3, 23.9)
- moved C11 0.98 mm to (39.2, 63.6)
- moved C29 0.89 mm to (32.9, 25.7)
- moved CN3 0.86 mm to (56.8, 23.4)
- moved CN2 0.85 mm to (66.4, 23.4)
- moved CN1 0.22 mm to (25.3, 66.0)
- moved C22 0.22 mm to (28.7, 39.5)
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Routing:
- net VBAT_BACKUP: track 13.7 -> 17.4 mm
- net GND: track 68.7 -> 65.1 mm, vias 164 -> 165
- net DFR0198: track 55.7 -> 57.7 mm
- net SEN0308: track 47.0 -> 48.7 mm
- net NRST: track 45.9 -> 47.2 mm
- net Net-(C29-Pad2): track 9.21 -> 10.1 mm
- net VSRC: track 11.6 -> 12.5 mm
- net VBAT: track 8.64 -> 9.49 mm
Other:
- board size 64.1 x 56.5 mm -> 64.1 x 59.3 mm
- board text added: "+"
- board text added: "-"
- board text added: "3.3V"
- board text added: "3V3_EXT"
- board text added: "BAT"
- board text added: "CR2032"
- board text added: "DFR"
- board text added: "GND"
- board text added: "HVOUT"
- board text added: "NRST"
- board text added: "PWR"
- board text added: "Prototipo PCB Main"
- board text added: "RX"
- board text added: "Reset"
- board text added: "SCL"
- board text added: "SDA"
- board text added: "SEN"
- board text added: "SRC"
- board text added: "SWCLK"
- board text added: "SWD"
- board text added: "SWDIO"
- board text added: "SWO"
- board text added: "TX"
- board text added: "USART"
- board text added: "USER"
- board text added: "VDD"
- board text added: "Vref"
- board text added: "islas cristales - OK plano 3.3V aislado de antena - OK vias debajo pads GND micros - OK antena como zona, no pista - OK cambiar pila holder - OK poner comentarios silkscreen - OK optimizar pistas"
- board text removed: "islas cristales - OK plano 3.3V aislado de antena - OK vias debajo pads GND micros - OK antena como zona, no pista - OK cambiar pila holder optimizar pistas poner comentarios silkscreen"

Commit message: pcb sent to jlcpcb
Parts:
- added CN10: Conn_01x03, Connector_PinHeader_2.54mm:PinHeader_1x03_P2.54mm_Vertical, F.Cu at (72.2, 62.7)
- added J2: Conn_01x02, Connector_PinHeader_2.54mm:PinHeader_1x02_P2.54mm_Vertical, F.Cu at (85.9, 56.5)
- added J3: Conn_01x02, Connector_PinHeader_2.54mm:PinHeader_1x02_P2.54mm_Vertical, F.Cu at (89.5, 56.5)
- R16, R17, R18: footprint Resistor_SMD:R_0402_1005Metric -> Resistor_SMD:R_0603_1608Metric
- moved SW1 24.7 mm to (41.2, 58.0)
- moved H1 24.2 mm to (39.1, 35.2)
- moved R16 24.1 mm to (43.9, 44.9)
- moved R17 24.1 mm to (43.9, 47.5)
- moved C5 24.1 mm to (80.3, 72.5)
- moved CN6 24.1 mm to (93.8, 79.6)
- moved CN8 24.1 mm to (74.0, 79.2)
- moved J1 24.1 mm to (75.2, 56.5)
- moved R6 24.1 mm to (81.8, 42.6)
- moved X2 24.1 mm to (64.1, 54.1)
- moved BT1 24.1 mm to (61.0, 68.6)
- moved L2 24.1 mm to (85.1, 64.7)
- moved L4 24.1 mm to (50.3, 51.4)
- moved R1 24.1 mm to (90.0, 46.1)
- moved R15 24.1 mm to (67.1, 49.0)
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Connections:
- CN6 pad 1: VDD_SENS -> DFR0198
- CN6 pad 2: DFR0198 -> GND
- CN6 pad 3: GND -> VDD_SENS
- CN7 pad 1: VDD_SENS -> SEN0308
- CN7 pad 2: SEN0308 -> VDD_SENS
- R1 pad 2: /Power Management/SRC -> /Power Management/SRC_INA
- R2 pad 2: /Power Management/BATT -> /Power Management/BATT_INA
- R5 pad 2: /Power Management/SRC -> /Power Management/SRC_INA
- R7 pad 2: /Power Management/BATT -> /Power Management/BATT_INA
Routing:
- net /Power Management/BATT_INA: track 0.00 -> 21.7 mm, vias 0 -> 1
- net /Power Management/SRC_INA: track 0.00 -> 10.7 mm, vias 0 -> 1
- net DFR0198: track 57.7 -> 63.9 mm
- net SEN0308: track 48.7 -> 54.8 mm
- net /Power Management/BATT: track 7.24 -> 2.62 mm, vias 2 -> 1
- net S0_AEM: track 35.4 -> 37.6 mm, vias 2 -> 1
- net GND: track 65.1 -> 63.6 mm, vias 165 -> 160
- net +3.3V: track 46.0 -> 47.4 mm
- net NRST: track 47.2 -> 45.8 mm
- net /Power Management/SRC: track 4.36 -> 3.17 mm, vias 2 -> 1
- net S1_AEM: track 36.4 -> 36.9 mm, vias 2 -> 1
- net /STM32WB55RG/VDDA: track 5.22 -> 5.75 mm
- net S2_AEM: vias 2 -> 1
Other:
- board text added: "S0"
- board text added: "S1"
- board text added: "S2"
