File: pcb/PCB Main/RF.kicad_sch (KiCad schematic)
At the start: 0 parts

Commit message: PCB casi lista
Parts:
- added C29: 1.2pF, Capacitor_SMD:C_0402_1005Metric, symbol Device:C
- added FLT1: Low_Pass_Filter_2.4GHz_50R, MLPF-WB55-01E3:MLPF-WB55-01E3, symbol MLPF-WB55-01E3:MLPF-WB55-01E3
- added L6: 3.6nH, LED_SMD:LED_0402_1005Metric, symbol Device:L
Connections:
- net RF1: now also FLT1.IN
- new net: FLT1.OUT, L6.1
- new net ANT: C29.2, L6.2
- new net GND: C29.1, FLT1.GND1, FLT1.GND2, FLT1.GND3, FLT1.GND4
Other:
- note added: "AN5165:"
- note added: "PCB Anthenna"
- note added: "RF"

Commit message: RF hecho
Other:
- moved on the sheet: C29, FLT1, L6

Commit message: vias pad GND
Parts:
- added C29: 1.2pF, Capacitor_SMD:C_0402_1005Metric, symbol Device:C
- renumbered C29 to C30
Connections:
- net GND: now also C29.1
- net at FLT1.OUT, L6.1: now also C29.2
Changed lines of the file:
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@@
+	)
+	(junction
+		(at 166.37 93.98)
+		(diameter 0)
+		(color 0 0 0 0)
 	)
 	(junction
@@
 	(wire
 		(pts
+			(xy 166.37 93.98) (xy 168.91 93.98)
+		)
+		(stroke
+			(width 0)
+			(type default)
+		)
+	)
+	(wire
+		(pts
 			(xy 149.86 104.14) (xy 149.86 106.68)
 		)
@@
 	(wire
 		(pts
-			(xy 148.59 93.98) (xy 168.91 93.98)
+			(xy 148.59 93.98) (xy 166.37 93.98)
 		)
 		(stroke
@@
 					(size 1.27 1.27)
 					(italic yes)
+				)
+			)
+		)
+	)
+	(symbol
+		(lib_id "Device:C")
+		(at 166.37 97.79 180)
+		(unit 1)
+		(exclude_from_sim no)
+		(in_bom yes)
+		(on_board yes)
+		(dnp yes)
+		(property "Reference" "C29"
+			(at 170.18 96.5199 0)
+			(effects
+				(font
+					(size 1.27 1.27)
+				)
+				(justify right)
+			)
+		)
+		(property "Value" "1.2pF"
+			(at 170.18 99.0599 0)
+			(effects
+				(font
+					(size 1.27 1.27)
+				)
+				(justify right)
+			)
+		)
+		(property "Footprint" "Capacitor_SMD:C_0402_1005Metric"
+			(at 165.4048 93.98 0)
+			(effects
+				(font
+					(size 1.27 1.27)
+				)
+				(hide yes)
+			)
+		)
+		(property "Datasheet" "~"
+			(at 166.37 97.79 0)
+			(effects
+				(font
+					(size 1.27 1.27)
+				)
+				(hide yes)
+			)
+		)
+		(property "Description" "1.2pF 50V C0G 0402 Multilayer Ceramic Capacitor SMD"
+			(at 166.37 97.79 0)
+			(effects
+				(font
+					(size 1.27 1.27)
+				)
+				(hide yes)
+			)
+		)
+		(property "Package" "0402"
+			(at 166.37 97.79 0)
+			(effects
+				(font
+					(size 1.27 1.27)
+				)
+				(hide yes)
+			)
+		)
+		(property "Manufacturer" "Murata Electronics"
+			(at 166.37 97.79 0)
+			(effects
+				(font
+					(size 1.27 1.27)
+				)
+				(hide yes)
+			)
+		)
+		(property "Supplier Part #" "C76899"
+			(at 166.37 97.79 0)
+			(effects
+				(font
+					(size 1.27 1.27)
+				)
+				(hide yes)
+			)
+		)
+		(property "Supplier" "JLCPCB"
+			(at 166.37 97.79 0)
+			(effects
+				(font
+					(size 1.27 1.27)
+				)
+				(hide yes)
+			)
+		)
+		(property "Supplier Part Type" "Extended"
+			(at 166.37 97.79 0)
+			(effects
+				(font
+					(size 1.27 1.27)
+				)
+				(hide yes)
+			)
+		)
+		(property "Component" "GJM1555C1H1R2WB01D"
+			(at 166.37 97.79 0)
+			(effects
+				(font
+					(size 1.27 1.27)
+				)
+				(hide yes)
+			)
+		)
+		(pin "2"
+		)
+		(pin "1"
+		)
+		(instances
+			(project "PCB Main"
+				(path "/9fa2563f-04cb-468b-9731-6177268fcdbf/ec8f88e8-78d2-4fac-b943-5ef9b1e2e231"
+					(reference "C29")
+					(unit 1)
 				)
 			)
@@
 	)
 	(symbol
+		(lib_id "power:GND")
+		(at 166.37 101.6 0)
+		(unit 1)
+		(exclude_from_sim no)
+		(in_bom yes)
+		(on_board yes)
+		(dnp no)
+		(fields_autoplaced yes)
+		(property "Reference" "#PWR062"
+			(at 166.37 107.95 0)
+			(effects
+				(font
+					(size 1.27 1.27)
+				)
+				(hide yes)
+			)
+		)
+		(property "Value" "GND"
+			(at 166.37 106.68 0)
+			(effects
+				(font
+					(size 1.27 1.27)
+				)
+			)
+		)
+		(property "Footprint" ""
+			(at 166.37 101.6 0)
+			(effects
+				(font
+					(size 1.27 1.27)
+				)
+				(hide yes)
+			)
+		)
+		(property "Datasheet" ""
+			(at 166.37 101.6 0)
+			(effects
+				(font
+					(size 1.27 1.27)
+				)
+				(hide yes)
+			)
+		)
+		(property "Description" "Power symbol creates a global label with name \"GND\" , ground"
+			(at 166.37 101.6 0)
+			(effects
+				(font
+					(size 1.27 1.27)
+				)
+				(hide yes)
+			)
+		)
+		(pin "1"
+		)
+		(instances
+			(project "PCB Main"
+				(path "/9fa2563f-04cb-468b-9731-6177268fcdbf/ec8f88e8-78d2-4fac-b943-5ef9b1e2e231"
+					(reference "#PWR062")
+					(unit 1)
+				)
+			)
+		)
+	)
+	(symbol
 		(lib_id "Device:L")
 		(at 172.72 93.98 90)
@@
 		(on_board yes)
 		(dnp no)
-		(property "Reference" "C29"
+		(property "Reference" "C30"
 			(at 182.88 96.5199 0)
 			(effects
@@
 			(project "PCB Main"
 				(path "/9fa2563f-04cb-468b-9731-6177268fcdbf/ec8f88e8-78d2-4fac-b943-5ef9b1e2e231"
-					(reference "C29")
+					(reference "C30")
 					(unit 1)
 				)

Commit message: pcb sent to jlcpcb
Parts:
- C29: now left out of the parts list
Other:
- moved on the sheet: C29
Changed lines of the file:
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@@
 	(symbol
 		(lib_id "Device:C")
-		(at 166.37 97.79 180)
+		(at 166.37 97.79 0)
+		(mirror x)
 		(unit 1)
 		(exclude_from_sim no)
-		(in_bom yes)
+		(in_bom no)
 		(on_board yes)
 		(dnp yes)
 		(property "Reference" "C29"
-			(at 170.18 96.5199 0)
+			(at 162.56 96.5199 0)
 			(effects
 				(font
@@
 		)
 		(property "Value" "1.2pF"
-			(at 170.18 99.0599 0)
+			(at 162.56 99.0599 0)
 			(effects
 				(font
@@
 		)
 		(property "Footprint" "Capacitor_SMD:C_0402_1005Metric"
-			(at 165.4048 93.98 0)
+			(at 167.3352 93.98 0)
 			(effects
 				(font
