File: pcb/PCB Main/PCB Main.kicad_sch (KiCad schematic)
At the start: 0 parts

Commit message: update
Changed lines of the file:
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@@
+		)
+	)
+	(text_box "TODO List"
+		(exclude_from_sim no)
+		(at 133.35 69.85 0)
+		(size 72.39 3.81)
+		(margins 0.9525 0.9525 0.9525 0.9525)
+		(stroke
+			(width 0)
+			(type solid)
+		)
+		(fill
+			(type color)
+			(color 255 229 191 1)
+		)
+		(effects
+			(font
+				(size 1.27 1.27)
+			)
+			(justify left top)
 		)
 	)
@@
 		(fill
 			(type color)
-			(color 255 255 194 1)
+			(color 255 229 191 1)
 		)
 		(effects
+			(font
+				(size 1.27 1.27)
+			)
+			(justify left top)
+		)
+	)
+	(text_box "- Upload method (USART or ST-LINK)\n- Upload power (if no battery)\n- RTC battery\n- Reset BTN\n- BLE\n- PV and BATT conection\n\n- Select components"
+		(exclude_from_sim no)
+		(at 133.35 74.93 0)
+		(size 72.39 34.29)
+		(margins 0.9525 0.9525 0.9525 0.9525)
+		(stroke
+			(width 0)
+			(type solid)
+		)
+		(fill
+			(type none)
+		)
+		(effects

Commit message: updates
Other:
- added sheet RF (RF.kicad_sch)
Changed lines of the file:
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@@
 		)
 	)
-	(text_box "Page 1 - Top Sheet\nPage 2 - STM32WB55RG\nPage 3 - Power Management"
+	(text_box "Page 1 - Top Sheet\nPage 2 - STM32WB55RG\nPage 3 - Power Management\nPage 4 - RF"
 		(exclude_from_sim no)
 		(at 25.4 74.93 0)
-		(size 101.6 7.62)
+		(size 101.6 10.16)
 		(margins 0.9525 0.9525 0.9525 0.9525)
 		(stroke
@@
 		)
 	)
-	(text_box "- Upload method (USART or ST-LINK)\n- Upload power (if no battery)\n- RTC battery\n- Reset BTN\n- BLE\n- PV and BATT conection\n\n- Select components"
+	(text_box "- Upload method (USART or ST-LINK): STLINK\n- Upload power (if no battery)\n- RTC battery\n- Reset BTN\n- BLE\n- PV and BATT conection\n\n- Select components"
 		(exclude_from_sim no)
 		(at 133.35 74.93 0)
@@
 	)
 	(sheet
-		(at 25.4 88.9)
+		(at 25.4 91.44)
 		(size 44.45 5.08)
 		(exclude_from_sim no)
@@
 		)
 		(property "Sheetname" "STM32WB55RG"
-			(at 25.4 88.1884 0)
+			(at 25.4 90.7284 0)
 			(effects
 				(font
@@
 		)
 		(property "Sheetfile" "STM32WB55RG.kicad_sch"
-			(at 25.4 94.5646 0)
+			(at 25.4 97.1046 0)
 			(effects
 				(font
@@
 	)
 	(sheet
-		(at 25.4 101.6)
+		(at 25.4 104.14)
 		(size 44.45 5.08)
 		(exclude_from_sim no)
@@
 		)
 		(property "Sheetname" "Power Management"
-			(at 25.4 100.8884 0)
+			(at 25.4 103.4284 0)
 			(effects
 				(font
@@
 		)
 		(property "Sheetfile" "Power Management.kicad_sch"
-			(at 25.4 107.2646 0)
+			(at 25.4 109.8046 0)
 			(effects
 				(font
@@
 				)
 			)
+		)
+	)
+	(sheet
+		(at 25.4 116.84)
+		(size 44.45 5.08)
+		(exclude_from_sim no)
+		(in_bom yes)
+		(on_board yes)
+		(dnp no)
+		(fields_autoplaced yes)
+		(stroke
+			(width 0.1524)
+			(type solid)
+		)
+		(fill
+			(color 0 0 0 0.0000)
+		)
+		(property "Sheetname" "RF"
+			(at 25.4 116.1284 0)
+			(effects
+				(font
+					(size 1.27 1.27)
+				)
+				(justify left bottom)
+			)
+		)
+		(property "Sheetfile" "RF.kicad_sch"
+			(at 25.4 122.5046 0)
+			(effects
+				(font
+					(size 1.27 1.27)
+				)
+				(justify left top)
+			)
+		)
+		(instances
+			(project "PCB Main"
+				(path "/9fa2563f-04cb-468b-9731-6177268fcdbf"
+					(page "4")
+				)
+			)

Commit message: PCB casi lista
Parts:
- added H1, H2, H3, H4: MountingHole, MountingHole:MountingHole_2.2mm_M2, symbol Mechanical:MountingHole
Other:
- added sheet External Connections (External Connections.kicad_sch)
- note added: "1-WIRE"
- note added: "3V3"
- note added: "Alerts"
- note added: "Analog"
- note added: "Anthenna"
- note added: "CR2032"
- note added: "HVOUT"
- note added: "I2C"
- note added: "IN1+"
- note added: "IN1-"
- note added: "IN2+"
- note added: "IN2-"
- note added: "IN3+"
- note added: "IN3-"
- note added: "SWD"
- note added: "Status"

Commit message: silkscreen
Other:
- moved on the sheet: H1, H2, H3, H4
Changed lines of the file:
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@@
-		)
-	)
-	(text_box "TODO List"
-		(exclude_from_sim no)
-		(at 17.78 105.41 0)
-		(size 83.82 3.81)
-		(margins 0.9525 0.9525 0.9525 0.9525)
-		(stroke
-			(width 0)
-			(type solid)
-		)
-		(fill
-			(type color)
-			(color 255 229 191 1)
-		)
-		(effects
-			(font
-				(size 1.27 1.27)
-			)
-			(justify left top)
 		)
 	)
@@
 		)
 	)
-	(text_box "- MOSFET para apagar sensores\n- BLE\n- Local storage: FRAM\n\n- PV and BATT connection\n\n- Select components"
-		(exclude_from_sim no)
-		(at 17.78 110.49 0)
-		(size 83.82 26.67)
-		(margins 0.9525 0.9525 0.9525 0.9525)
-		(stroke
-			(width 0)
-			(type solid)
-		)
-		(fill
-			(type none)
-		)
-		(effects
-			(font
-				(size 1.27 1.27)
-			)
-			(justify left top)
-		)
-	)
 	(text_box "Main Battery"
 		(exclude_from_sim no)
@@
 	(symbol
 		(lib_id "Mechanical:MountingHole")
-		(at 24.13 148.59 0)
+		(at 25.4 110.49 0)
 		(unit 1)
 		(exclude_from_sim no)
@@
 		(fields_autoplaced yes)
 		(property "Reference" "H1"
-			(at 26.67 147.3199 0)
+			(at 27.94 109.2199 0)
 			(effects
 				(font
@@
 		)
 		(property "Value" "MountingHole"
-			(at 26.67 149.8599 0)
+			(at 27.94 111.7599 0)
 			(effects
 				(font
@@
 		)
 		(property "Footprint" "MountingHole:MountingHole_2.2mm_M2"
-			(at 24.13 148.59 0)
+			(at 25.4 110.49 0)
 			(effects
 				(font
@@
 		)
 		(property "Datasheet" "~"
-			(at 24.13 148.59 0)
+			(at 25.4 110.49 0)
 			(effects
 				(font
@@
 		)
 		(property "Description" "Mounting Hole M2"
-			(at 24.13 148.59 0)
+			(at 25.4 110.49 0)
 			(effects
 				(font
@@
 		)
 		(property "Manufacturer" "-"
-			(at 24.13 148.59 0)
+			(at 25.4 110.49 0)
 			(effects
 				(font
@@
 		)
 		(property "Package" "NPTH"
-			(at 24.13 148.59 0)
+			(at 25.4 110.49 0)
 			(effects
 				(font
@@
 		)
 		(property "Supplier" "-"
-			(at 24.13 148.59 0)
+			(at 25.4 110.49 0)
 			(effects
 				(font
@@
 		)
 		(property "Supplier Part #" "-"
-			(at 24.13 148.59 0)
+			(at 25.4 110.49 0)
 			(effects
 				(font
@@
 		)
 		(property "Supplier Part Type" "-"
-			(at 24.13 148.59 0)
+			(at 25.4 110.49 0)
 			(effects
 				(font
@@
 	(symbol
 		(lib_id "Mechanical:MountingHole")
-		(at 24.13 167.64 0)
+		(at 25.4 129.54 0)
 		(unit 1)
 		(exclude_from_sim no)
@@
 		(fields_autoplaced yes)
 		(property "Reference" "H4"
-			(at 26.67 166.3699 0)
+			(at 27.94 128.2699 0)
 			(effects
 				(font
@@
 		)
 		(property "Value" "MountingHole"
-			(at 26.67 168.9099 0)
+			(at 27.94 130.8099 0)
 			(effects
 				(font
@@
 		)
 		(property "Footprint" "MountingHole:MountingHole_2.2mm_M2"
-			(at 24.13 167.64 0)
+			(at 25.4 129.54 0)
 			(effects
 				(font
@@
 		)
 		(property "Datasheet" "~"
-			(at 24.13 167.64 0)
+			(at 25.4 129.54 0)
 			(effects
 				(font
@@
 		)
 		(property "Description" "Mounting Hole M2"
-			(at 24.13 167.64 0)
+			(at 25.4 129.54 0)
 			(effects
 				(font
@@
 		)
 		(property "Manufacturer" "-"
-			(at 24.13 167.64 0)
+			(at 25.4 129.54 0)
 			(effects
 				(font
@@
 		)
 		(property "Package" "NPTH"
-			(at 24.13 167.64 0)
+			(at 25.4 129.54 0)
 			(effects
 				(font
@@
 		)
 		(property "Supplier" "-"
-			(at 24.13 167.64 0)
+			(at 25.4 129.54 0)
 			(effects
 				(font
@@
 		)
 		(property "Supplier Part #" "-"
-			(at 24.13 167.64 0)
+			(at 25.4 129.54 0)
 			(effects
 				(font
@@
 		)
 		(property "Supplier Part Type" "-"
-			(at 24.13 167.64 0)
+			(at 25.4 129.54 0)
 			(effects
 				(font
@@
 	(symbol
 		(lib_id "Mechanical:MountingHole")
-		(at 24.13 161.29 0)
+		(at 25.4 123.19 0)
 		(unit 1)
 		(exclude_from_sim no)
@@
 		(fields_autoplaced yes)
 		(property "Reference" "H3"
-			(at 26.67 160.0199 0)
+			(at 27.94 121.9199 0)
 			(effects
 				(font
@@
 		)
 		(property "Value" "MountingHole"
-			(at 26.67 162.5599 0)
+			(at 27.94 124.4599 0)
 			(effects
 				(font
@@
 		)
 		(property "Footprint" "MountingHole:MountingHole_2.2mm_M2"
-			(at 24.13 161.29 0)
+			(at 25.4 123.19 0)
 			(effects
 				(font
@@
 		)
 		(property "Datasheet" "~"
-			(at 24.13 161.29 0)
+			(at 25.4 123.19 0)
 			(effects
 				(font
@@
 		)
 		(property "Description" "Mounting Hole M2"
-			(at 24.13 161.29 0)
+			(at 25.4 123.19 0)
 			(effects
 				(font
@@
 		)
 		(property "Manufacturer" "-"
-			(at 24.13 161.29 0)
+			(at 25.4 123.19 0)
 			(effects
 				(font
@@
 		)
 		(property "Package" "NPTH"
-			(at 24.13 161.29 0)
+			(at 25.4 123.19 0)
 			(effects
 				(font
@@
 		)
 		(property "Supplier" "-"
-			(at 24.13 161.29 0)
+			(at 25.4 123.19 0)
 			(effects
 				(font
@@
 		)
 		(property "Supplier Part #" "-"
-			(at 24.13 161.29 0)
+			(at 25.4 123.19 0)
 			(effects
 				(font
@@
 		)
 		(property "Supplier Part Type" "-"
-			(at 24.13 161.29 0)
+			(at 25.4 123.19 0)
 			(effects
 				(font
@@
 	(symbol
 		(lib_id "Mechanical:MountingHole")
-		(at 24.13 154.94 0)
+		(at 25.4 116.84 0)
 		(unit 1)
 		(exclude_from_sim no)
@@
 		(fields_autoplaced yes)
 		(property "Reference" "H2"
-			(at 26.67 153.6699 0)
+			(at 27.94 115.5699 0)
 			(effects
 				(font
@@
 		)
 		(property "Value" "MountingHole"
-			(at 26.67 156.2099 0)
+			(at 27.94 118.1099 0)
 			(effects
 				(font
@@
 		)
 		(property "Footprint" "MountingHole:MountingHole_2.2mm_M2"
-			(at 24.13 154.94 0)
+			(at 25.4 116.84 0)
 			(effects
 				(font
@@
 		)
 		(property "Datasheet" "~"
-			(at 24.13 154.94 0)
+			(at 25.4 116.84 0)
 			(effects
 				(font
@@
 		)
 		(property "Description" "Mounting Hole M2"
-			(at 24.13 154.94 0)
+			(at 25.4 116.84 0)
 			(effects
 				(font
@@
 		)
 		(property "Manufacturer" "-"
-			(at 24.13 154.94 0)
+			(at 25.4 116.84 0)
 			(effects
 				(font
@@
 		)
 		(property "Package" "NPTH"
-			(at 24.13 154.94 0)
+			(at 25.4 116.84 0)
 			(effects
 				(font
@@
 		)
 		(property "Supplier" "-"
-			(at 24.13 154.94 0)
+			(at 25.4 116.84 0)
 			(effects
 				(font
@@
 		)
 		(property "Supplier Part #" "-"
-			(at 24.13 154.94 0)
+			(at 25.4 116.84 0)
 			(effects
 				(font
@@
 		)
 		(property "Supplier Part Type" "-"
-			(at 24.13 154.94 0)
-			(effects
-				(font
+			(at 25.4 116.84 0)
+			(effects
+				(font

Commit message: pcb sent to jlcpcb
Parts:
- H1, H2, H3, H4: Component (none) -> -
Changed lines of the file:
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@@
+			)
+		)
+		(property "Component" "-"
+			(at 25.4 110.49 0)
+			(effects
+				(font
+					(size 1.27 1.27)
+				)
+				(hide yes)
 			)
 		)
@@
 			)
 		)
+		(property "Component" "-"
+			(at 25.4 129.54 0)
+			(effects
+				(font
+					(size 1.27 1.27)
+				)
+				(hide yes)
+			)
+		)
 		(instances
 			(project "PCB Main"
@@
 			)
 		)
+		(property "Component" "-"
+			(at 25.4 123.19 0)
+			(effects
+				(font
+					(size 1.27 1.27)
+				)
+				(hide yes)
+			)
+		)
 		(instances
 			(project "PCB Main"
@@
 			(at 25.4 116.84 0)
 			(effects
+				(font
+					(size 1.27 1.27)
+				)
+				(hide yes)
+			)
+		)
+		(property "Component" "-"
+			(at 25.4 116.84 0)
+			(effects

Commit message: cambios :)
Other:
- note added: "SPI"
