File: pcb/PCB Main/Power Management.kicad_sch (KiCad schematic)
At the start: 28 parts, among them J1 Conn_02x02_Odd_Even, J2 Conn_01x02, U2 AEM10941, U3 INA3221

Commit message: update
Parts:
- removed C11, C12, C13: 100uF, symbol Device:C
- removed J1: Conn_02x02_Odd_Even, Connector_PinHeader_1.27mm:PinHeader_2x02_P1.27mm_Vertical, symbol Connector_Generic:Conn_02x02_Odd_Even
- added J1: Conn_01x03, Connector_PinHeader_2.54mm:PinHeader_1x03_P2.54mm_Vertical, symbol Connector_Generic:Conn_01x03
- added J3, J4: Conn_01x02, Connector_PinHeader_1.27mm:PinHeader_1x02_P1.27mm_Vertical, symbol Connector_Generic:Conn_01x02
- added JP1: Jumper_01x02_P2.54mm, symbol PZG_Jumpers:Jumper_01x02_2.54
- C1: Component (none) -> CC0603KRX7R9BB104; Componente CC0603KRX7R9BB104 -> (none); Manufacturer (none) -> YAGEO; Package (none) -> C_0603; Supplier (none) -> JLCPCB; Supplier Part # (none) -> C14663
- C10: value 100uF -> 10uF; footprint (none) -> Capacitor_SMD:C_0805_2012Metric; Component (none) -> GRM21BR71A106KE51L; Manufacturer (none) -> Murata Electronics; Package (none) -> C_0805; Supplier (none) -> JLCPCB; Supplier Part # (none) -> C86038
- C2, C3, C4: Component (none) -> CC0603KRX7R9BB333; Componente CC0603KRX7R9BB333 -> (none); Manufacturer (none) -> YAGEO; Package (none) -> C_0603; Supplier (none) -> JLCPCB; Supplier Part # (none) -> C106856
- C5, C6, C8: Component (none) -> GRM21BR71A106KE51L; Componente GRM21BR71A106KE51L -> (none); Manufacturer (none) -> Murata Electronics; Package (none) -> C_0805; Supplier (none) -> JLCPCB; Supplier Part # (none) -> C86038
- C7: Component (none) -> GRM21BZ71A226ME15L; Componente GRM21BZ71A226ME15L -> (none); Manufacturer (none) -> Murata Electronics; Package (none) -> C_0805; Supplier (none) -> JLCPCB; Supplier Part # (none) -> C907991
- C9: value 150uF -> 220uF; footprint Capacitor_SMD:C_1206_3216Metric -> Capacitor_SMD:CP_Elec_8x6.2; Component (none) -> EEEFK1A221P; Manufacturer (none) -> PANASONIC; Package (none) -> SMD (8x6.2); Supplier (none) -> JLCPCB; Supplier Part # (none) -> C401648
- J2: footprint Connector_PinHeader_1.27mm:PinHeader_1x02_P1.27mm_Vertical -> Connector_PinHeader_2.54mm:PinHeader_1x02_P2.54mm_Vertical
- L1: Component (none) -> LPS4018-103MRC; Componente LPS4018-103MRC -> (none); Manufacturer (none) -> Coilcraft; Package (none) -> SMD (3.9x3.9); Supplier (none) -> JLCPCB; Supplier Part # (none) -> C6127589
- L2: Component (none) -> MLZ2012N100LT000; Componente MLZ2012N100LT000 -> (none); Manufacturer (none) -> TDK; Package (none) -> L_0805; Supplier (none) -> JLCPCB; Supplier Part # (none) -> C88182
- R1, R2, R3: Component (none) -> CSRN2512FTR100; Componente CSRN2512FTR100 -> (none); Manufacturer (none) -> SEI(Stackpole Elec); Package (none) -> R_2512; Supplier (none) -> JLCPCB; Supplier Part # (none) -> C346817
- R4, R5, R6, R7, R8, R9: Component (none) -> RC0603FR-0710RL; Componente RC0603FR-0710RL -> (none); Manufacturer (none) -> YAGEO; Package (none) -> R_0603; Supplier (none) -> JLCPCB; Supplier Part # (none) -> C109318
- U2: Component (none) -> AEM10941-QFN; Componente AEM10941-QFN -> (none); Manufacturer (none) -> e-peas; Package (none) -> QFN-28
- U3: Component (none) -> INA3221AIRGVR; Componente INA3221AIRGVR -> (none); Manufacturer (none) -> Texas Instruments; Package (none) -> QFN-16-EP (4x4); Supplier (none) -> JLCPCB; Supplier Part # (none) -> C181255
Connections:
- net BAT- is gone; now on net BATT: R2.2, R7.2
- net LOAD+ is gone; now on net HVOUT: R3.1, R8.2
- net PV- is gone; now on net SRC: R1.2, R5.2
- net 3V3_EXT: now also J1.1 (Pin_1)
- net BAT+: now also J4.1 (Pin_1)
- net BATT: now also C10.1, C9.2; no longer C9.1
- net BUCK: now also C6.1; no longer C6.2
- net GND: now also C10.2, C6.2, C8.1, C9.1, J3.2 (Pin_2), J4.2 (Pin_2); no longer C10.1, C6.1, C8.2, C9.2
- net HVOUT: now also C8.2, J1.3 (Pin_3); no longer C8.1
- net PV+: now also J3.1 (Pin_1)
- net LOAD- renamed 3V3
- net VDD renamed +3.3V
- net +3.3V: now also J1.2 (Pin_2); no longer C10.2
Other:
- note added: "Colocar pila CR2032 o similar para alimentar RTC cuando no hay HVOUT"
- note added: "Comprobar valores de capacitores"
- note added: "Mirar conectores correctos"
- note added: "POWER MEASURING"
- note added: "Pensar en otras alternativas para alimentar al STM32 si no hay HVOUT para subir codigo"
- note added: "Pin max voltages and currents"
- note removed: "MCU POWER"
- note removed: "POWER SENSING"
- note removed: "Pensar en otras alternativas"
- moved on the sheet: C5, C7, C9, L1, L2, U2

Commit message: updates
Changed lines of the file:
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@@
 	(text "Configurar MPPT"
 		(exclude_from_sim no)
-		(at 55.88 87.63 0)
+		(at 71.12 99.06 0)
 		(effects
 			(font
@@
 		(exclude_from_sim no)
 		(at 121.92 73.66 0)
-		(size 34.29 7.62)
+		(size 33.02 7.62)
 		(margins 0.9525 0.9525 0.9525 0.9525)
 		(stroke
@@
 		)
 	)
+	(text_box "C5: CSRC\nC6: CBOOST\nC7: CBUCK\nC8: CHV\nC9: CBATT\n\nL1: LBOOST\nL2: LBUCK"
+		(exclude_from_sim no)
+		(at 34.29 81.28 0)
+		(size 15.24 17.78)
+		(margins 0.9525 0.9525 0.9525 0.9525)
+		(stroke
+			(width 0)
+			(type solid)
+		)
+		(fill
+			(type color)
+			(color 255 229 191 1)
+		)
+		(effects
+			(font
+				(size 1.27 1.27)
+			)
+			(justify left top)
+		)
+	)
 	(text_box "HVOUT is 3.3V when BATT is "
 		(exclude_from_sim no)
 		(at 121.92 85.09 0)
-		(size 34.29 12.7)
+		(size 33.02 12.7)
 		(margins 0.9525 0.9525 0.9525 0.9525)
 		(stroke
@@
 		(property "Intersheetrefs" "${INTERSHEET_REFS}"
 			(at 118.4342 72.39 0)
-			(effects
-				(font
-					(size 1.27 1.27)
-				)
-				(justify left)
-				(hide yes)
-			)
-		)
-	)
-	(global_label "VBAT"
-		(shape output)
-		(at 224.79 58.42 0)
-		(fields_autoplaced yes)
-		(effects
-			(font
-				(size 1.27 1.27)
-			)
-			(justify left)
-		)
-		(property "Intersheetrefs" "${INTERSHEET_REFS}"
-			(at 232.19 58.42 0)
 			(effects
 				(font
@@
 					(unit 1)
 				)
+			)
+		)
+	)
+	(symbol
+		(lib_id "power:+3.3V")
+		(at 226.06 58.42 0)
+		(unit 1)
+		(exclude_from_sim no)
+		(in_bom yes)
+		(on_board yes)
+		(dnp no)
+		(fields_autoplaced yes)
+		(property "Reference" "#PWR048"
+			(at 226.06 62.23 0)
+			(effects
+				(font
+					(size 1.27 1.27)
+				)
+				(hide yes)
+			)
+		)
+		(property "Value" "VBATT"
+			(at 226.06 53.34 0)
+			(effects
+				(font
+					(size 1.27 1.27)
+				)
+			)
+		)
+		(property "Footprint" ""
+			(at 226.06 58.42 0)
+			(effects
+				(font
+					(size 1.27 1.27)
+				)
+				(hide yes)
+			)
+		)
+		(property "Datasheet" ""
+			(at 226.06 58.42 0)
+			(effects
+				(font
+					(size 1.27 1.27)
+				)
+				(hide yes)
+			)
+		)
+		(property "Description" "Power symbol creates a global label with name \"+3.3V\""
+			(at 226.06 58.42 0)
+			(effects
+				(font
+					(size 1.27 1.27)
+				)
+				(hide yes)
+			)
+		)
+		(pin "1"
+		)
+		(instances
+			(project "PCB Main"
+				(path "/9fa2563f-04cb-468b-9731-6177268fcdbf/b888a684-3263-4153-9730-9658fff4b3b0"
+					(reference "#PWR048")
+					(unit 1)
+				)

Commit message: PCB casi lista
Parts:
- removed C10: 10uF, Capacitor_SMD:C_0805_2012Metric, symbol Device:C
- removed J2: Conn_01x02, Connector_PinHeader_2.54mm:PinHeader_1x02_P2.54mm_Vertical, symbol Connector_Generic:Conn_01x02
- removed J3, J4: Conn_01x02, Connector_PinHeader_1.27mm:PinHeader_1x02_P1.27mm_Vertical, symbol Connector_Generic:Conn_01x02
- added Q1: AO3401A, Package_TO_SOT_SMD:SOT-23, symbol Transistor_FET:AO3401A
- added R10, R11, R12: 10k, Resistor_SMD:R_0402_1005Metric, symbol Device:R
- added R18: 100k, Resistor_SMD:R_0402_1005Metric, symbol Device:R
- C1: value 0.1uF -> 100nF; footprint Capacitor_SMD:C_0603_1608Metric -> Capacitor_SMD:C_0402_1005Metric; Component CC0603KRX7R9BB104 -> CL05B104KO5NNNC; Manufacturer YAGEO -> Samsung; Package C_0603 -> 0402; Supplier Part # C14663 -> C1525; Supplier Part Type (none) -> Basic
- C2, C3, C4: value 33nF -> 100nF; footprint Capacitor_SMD:C_0603_1608Metric -> Capacitor_SMD:C_0402_1005Metric; Component CC0603KRX7R9BB333 -> CL05B104KO5NNNC; Manufacturer YAGEO -> Samsung; Package C_0603 -> 0402; Supplier Part # C106856 -> C1525; Supplier Part Type (none) -> Basic
- C5, C6, C8: footprint Capacitor_SMD:C_0805_2012Metric -> Capacitor_SMD:C_0603_1608Metric; Component GRM21BR71A106KE51L -> CL10A106KP8NNNC; Manufacturer Murata Electronics -> Samsung; Package C_0805 -> 0603; Supplier Part # C86038 -> C19702; Supplier Part Type (none) -> Basic
- C7: footprint Capacitor_SMD:C_0805_2012Metric -> Capacitor_SMD:C_0603_1608Metric; Component GRM21BZ71A226ME15L -> CL10A226MQ8NRNC; Manufacturer Murata Electronics -> Samsung; Package C_0805 -> 0603; Supplier Part # C907991 -> C59461; Supplier Part Type (none) -> Basic
- C9: value 220uF -> 150uF; footprint Capacitor_SMD:CP_Elec_8x6.2 -> Capacitor_SMD:C_1206_3216Metric; Component EEEFK1A221P -> GRM31CR60J157ME11L; Manufacturer PANASONIC -> Murata Electronics; Package SMD (8x6.2) -> 1206; Supplier Part # C401648 -> C528968; Supplier Part Type (none) -> Extended
- J1: Supplier Part Type (none) -> -
- JP1: Supplier Part Type (none) -> Mechanical Assembly
- L1: Package SMD (3.9x3.9) -> SMD 3.9x3.9mm; Supplier Part Type (none) -> Extended
- L2: footprint Inductor_SMD:L_0805_2012Metric -> Inductor_SMD:L_0603_1608Metric; Component MLZ2012N100LT000 -> MLZ1608M100WT000; Package L_0805 -> 0603; Supplier Part # C88182 -> C76798; Supplier Part Type (none) -> Extended
- R1, R2, R3: value 0.1 -> 0.33; Component CSRN2512FTR100 -> RLP25FEER330; Manufacturer SEI(Stackpole Elec) -> TA-I Tech; Package R_2512 -> 2512; Supplier Part # C346817 -> C393076; Supplier Part Type (none) -> Extended
- R4, R5, R6, R7, R8, R9: footprint Resistor_SMD:R_0603_1608Metric -> Resistor_SMD:R_0402_1005Metric; Component RC0603FR-0710RL -> 0402WGF100JTCE; Manufacturer YAGEO -> UNI-ROYAL; Package R_0603 -> 0402; Supplier Part # C109318 -> C25077; Supplier Part Type (none) -> Basic
- U2: Supplier (none) -> Mouser; Supplier Part # (none) -> 120-AEM10941-QFN; Supplier Part Type (none) -> -
- U3: Supplier Part Type (none) -> Extended
Connections:
- net +3.3V: now also R3.2, R9.2, U3.16 (VPU), Q1.2 (S), R10.1, R11.1, R12.1, R18.1; no longer J1.2 (Pin_2)
- net 3V3: now also J1.2 (Pin_2), R3.1, R8.2; no longer R3.2, R9.2
- net BATT: now also C9.1; no longer C9.2
- net GND: now also C9.2; no longer C9.1
- net HVOUT: no longer R3.1, R8.2
- net SRC: now also U2.26 (FB_COLD)
- net PV_INA: now reaches U3.10 (PV)
- net PV_INA: now also R10.2
- net WAR_INA: now reaches U3.8 (WARNING)
- net WAR_INA: now also R12.2
- net CRI_INA: now reaches U3.9 (CRITICAL)
- net CRI_INA: now also R11.2
- net at C5.1, U2.27 (BUFSRC): now also L1.2; no longer L1.1
- net at U2.28 (SWBOOST): now also L1.1; no longer L1.2
- net BAT+ renamed VBAT
- net PV+ renamed VSRC
- net S0 renamed S0_AEM
- net S1 renamed S1_AEM
- net S2 renamed S2_AEM
- new net GATE_SENS: Q1.1 (G), R18.2
- new net VDD_SENS: Q1.3 (D)
- no-connect marks 12 -> 7
Other:
- note added: "3.3V BUS SWITCHING"
- note added: "SENSOR SUPPLY SWITCH"
- note removed: "Colocar pila CR2032 o similar para alimentar RTC cuando no hay HVOUT"
- note removed: "Comprobar valores de capacitores"
- note removed: "Mirar conectores correctos"
- note removed: "Pensar en otras alternativas para alimentar al STM32 si no hay HVOUT para subir codigo"
- moved on the sheet: C1, C2, C3, C4, C5, C6, C7, C8, J1, JP1, L1, L2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

Commit message: retoques
Parts:
- R1, R2, R3: value 0.33 -> 0.22; Component RLP25FEER330 -> RLP25FEER220; Supplier Part # C393076 -> C912987
Changed lines of the file:
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@@
 			)
 		)
-		(property "Value" "0.33"
+		(property "Value" "0.22"
 			(at 50.8 151.1299 0)
 			(effects
@@
 			)
 		)
-		(property "Description" "330mΩ 2W Current Sense Resistor ±1% ±50ppm/℃ 2512 SMD"
+		(property "Description" "220mΩ 2W Current Sense Resistor ±1% ±50ppm/℃ 2512 SMD"
 			(at 48.26 149.86 0)
 			(effects
@@
 			)
 		)
-		(property "Component" "RLP25FEER330"
+		(property "Component" "RLP25FEER220"
 			(at 48.26 149.86 0)
 			(effects
@@
 			)
 		)
-		(property "Supplier Part #" "C393076"
+		(property "Supplier Part #" "C912987"
 			(at 48.26 149.86 0)
 			(effects
@@
 			)
 		)
-		(property "Value" "0.33"
+		(property "Value" "0.22"
 			(at 50.8 171.4499 0)
 			(effects
@@
 			)
 		)
-		(property "Description" "330mΩ 2W Current Sense Resistor ±1% ±50ppm/℃ 2512 SMD"
+		(property "Description" "220mΩ 2W Current Sense Resistor ±1% ±50ppm/℃ 2512 SMD"
 			(at 48.26 170.18 0)
 			(effects
@@
 			)
 		)
-		(property "Component" "RLP25FEER330"
+		(property "Component" "RLP25FEER220"
 			(at 48.26 170.18 0)
 			(effects
@@
 			)
 		)
-		(property "Supplier Part #" "C393076"
+		(property "Supplier Part #" "C912987"
 			(at 48.26 170.18 0)
 			(effects
@@
 			)
 		)
-		(property "Value" "0.33"
+		(property "Value" "0.22"
 			(at 50.8 130.8099 0)
 			(effects
@@
 			)
 		)
-		(property "Description" "330mΩ 2W Current Sense Resistor ±1% ±50ppm/℃ 2512 SMD"
+		(property "Description" "220mΩ 2W Current Sense Resistor ±1% ±50ppm/℃ 2512 SMD"
 			(at 48.26 129.54 0)
 			(effects
@@
 			)
 		)
-		(property "Component" "RLP25FEER330"
+		(property "Component" "RLP25FEER220"
 			(at 48.26 129.54 0)
 			(effects
@@
 			)
 		)
-		(property "Supplier Part #" "C393076"
+		(property "Supplier Part #" "C912987"
 			(at 48.26 129.54 0)
 			(effects

Commit message: pcb sent to jlcpcb
Parts:
- added CN10: Conn_01x03, Connector_PinHeader_2.54mm:PinHeader_1x03_P2.54mm_Vertical, symbol Connector_Generic:Conn_01x03
- added J2, J3: Conn_01x02, Connector_PinHeader_2.54mm:PinHeader_1x02_P2.54mm_Vertical, symbol Connector_Generic:Conn_01x02
- added JP2, JP3: Jumper_01x02_P2.54mm, symbol PZG_Jumpers:Jumper_01x02_2.54
- J1: Package (none) -> PTH; now left out of the parts list
- JP1: now left out of the parts list
- R18: footprint Resistor_SMD:R_0402_1005Metric -> Resistor_SMD:R_0603_1608Metric; Component 0402WGF1003TCE -> 0603WAF1003T5E; Package 0402 -> 0603; Supplier Part # C25741 -> C25803
- U2: Supplier Mouser -> JLCPCB; Supplier Part # 120-AEM10941-QFN -> C9900027046; Supplier Part Type - -> Extended
Connections:
- net BATT: now also J2.2 (Pin_2); no longer R2.2, R7.2
- net S0_AEM: now also CN10.3 (Pin_3)
- net S1_AEM: now also CN10.2 (Pin_2)
- net S2_AEM: now also CN10.1 (Pin_1)
- net SRC: now also J3.2 (Pin_2); no longer R1.2, R5.2
- new net BATT_INA: J2.1 (Pin_1), R2.2, R7.2
- new net SRC_INA: J3.1 (Pin_1), R1.2, R5.2

Commit message: cambios :)
Other:
- note removed: "Configurar MPPT"
- moved on the sheet: CN10
Changed lines of the file:
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@@
 		)
 	)
-	(text "Configurar MPPT"
-		(exclude_from_sim no)
-		(at 62.23 97.79 0)
-		(effects
-			(font
-				(size 1.27 1.27)
-			)
-			(justify bottom)
-		)
-	)
 	(text "3.3V BUS SWITCHING"
 		(exclude_from_sim no)
@@
 		)
 	)
-	(text_box "C5: CSRC\nC6: CBOOST\nC7: CBUCK\nC8: CHV\nC9: CBATT\n\nL1: LBOOST\nL2: LBUCK"
+	(text_box "C5: CSRC\nC6: CBUCK\nC7: CBOOST\nC8: CHV\nC9: CBATT\n\nL1: LBOOST\nL2: LBUCK"
 		(exclude_from_sim no)
 		(at 139.7 27.94 0)
@@
 	(wire
 		(pts
-			(xy 233.68 86.36) (xy 236.22 86.36)
+			(xy 251.46 44.45) (xy 254 44.45)
 		)
 		(stroke
@@
 	(wire
 		(pts
-			(xy 233.68 88.9) (xy 236.22 88.9)
+			(xy 251.46 46.99) (xy 254 46.99)
 		)
 		(stroke
@@
 	(wire
 		(pts
-			(xy 233.68 91.44) (xy 236.22 91.44)
+			(xy 251.46 49.53) (xy 254 49.53)
 		)
 		(stroke
@@
 	(global_label "S1_AEM"
 		(shape bidirectional)
-		(at 236.22 88.9 0)
+		(at 254 46.99 0)
 		(fields_autoplaced yes)
 		(effects
@@
 		)
 		(property "Intersheetrefs" "${INTERSHEET_REFS}"
-			(at 247.3921 88.9 0)
+			(at 265.1721 46.99 0)
 			(effects
 				(font
@@
 	(global_label "S2_AEM"
 		(shape bidirectional)
-		(at 236.22 86.36 0)
+		(at 254 44.45 0)
 		(fields_autoplaced yes)
 		(effects
@@
 		)
 		(property "Intersheetrefs" "${INTERSHEET_REFS}"
-			(at 247.3921 86.36 0)
+			(at 265.1721 44.45 0)
 			(effects
 				(font
@@
 	(global_label "S0_AEM"
 		(shape bidirectional)
-		(at 236.22 91.44 0)
+		(at 254 49.53 0)
 		(fields_autoplaced yes)
 		(effects
@@
 		)
 		(property "Intersheetrefs" "${INTERSHEET_REFS}"
-			(at 247.3921 91.44 0)
+			(at 265.1721 49.53 0)
 			(effects
 				(font
@@
 	(symbol
 		(lib_id "Connector_Generic:Conn_01x03")
-		(at 228.6 88.9 0)
+		(at 246.38 46.99 0)
 		(mirror y)
 		(unit 1)
@@
 		(fields_autoplaced yes)
 		(property "Reference" "CN10"
-			(at 228.6 80.01 0)
+			(at 246.38 38.1 0)
 			(effects
 				(font
@@
 		)
 		(property "Value" "Conn_01x03"
-			(at 228.6 82.55 0)
+			(at 246.38 40.64 0)
 			(effects
 				(font
@@
 		)
 		(property "Footprint" "Connector_PinHeader_2.54mm:PinHeader_1x03_P2.54mm_Vertical"
-			(at 228.6 88.9 0)
+			(at 246.38 46.99 0)
 			(effects
 				(font
@@
 		)
 		(property "Datasheet" "~"
-			(at 228.6 88.9 0)
+			(at 246.38 46.99 0)
 			(effects
 				(font
@@
 		)
 		(property "Description" "01x03 2.54mm Pin Header Vertical"
-			(at 228.6 88.9 0)
+			(at 246.38 46.99 0)
 			(effects
 				(font
@@
 		)
 		(property "Supplier Part Type" "-"
-			(at 228.6 88.9 0)
+			(at 246.38 46.99 0)
 			(effects
 				(font
@@
 		)
 		(property "Package" "PTH"
-			(at 228.6 88.9 0)
+			(at 246.38 46.99 0)
 			(effects
 				(font
