File: pcb/PCB Main/STM32WB55RG.kicad_sch (KiCad schematic)
At the start: 16 parts, among them CN1 Conn_ARM_JTAG_SWD_10, U1 STM32WB55RGVx, Y1 HSE, Y2 LSE

Commit message: update
Parts:
- added C11, C12, C13, C14: 100uF, symbol Device:C
- added D1: BAT54J, Diode_SMD:D_SOD-323F, symbol Diode:BAT54J
- added LED1: GREEN, LED_SMD:LED_0603_1608Metric, symbol Device:LED
- added LED2: BLUE, LED_SMD:LED_0603_1608Metric, symbol Device:LED
- added R11, R12: 1k, symbol Device:R
- L3: footprint (none) -> Inductor_SMD:L_0603_1608Metric; Component (none) -> FCM1608KF-601T02; Componente FCM1608KF-601T02 -> (none); Manufacturer (none) -> TAI-TECH; Package (none) -> L_0603; Supplier (none) -> JLCPCB; Supplier Part # (none) -> C127281
- U1: Component (none) -> STM32WB55RGV6; Manufacturer (none) -> STMicroelectronics; Package (none) -> QFN-68-EP (8x8); Supplier (none) -> JLCPCB; Supplier Part # (none) -> C401505
- Y1: value HSE -> 32MHz; Component (none) -> NX2016SA-32M-EXS00A-CS06465; Componente NX2016SA-32M-EXS00A-CS06465 -> (none); Manufacturer (none) -> NDK; Package (none) -> SMD2016-4P; Supplier (none) -> JLCPCB; Supplier Part # (none) -> C1986260
- Y2: value LSE -> 32.768kHz; Component (none) -> NX2012SA-32.768KHZ-STD-MUB-2; Componente NX2012SA-32.768KHZ-STD-MUB-2 -> (none); Manufacturer (none) -> NDK; Package (none) -> SMD2012-2P; Supplier (none) -> JLCPCB; Supplier Part # (none) -> C891748
- renumbered C14 to C15, C15 to C16, C16 to C17, C17 to C18, C18 to C19, C19 to C20, C20 to C21, C21 to C22, C22 to C23
Connections:
- net GND: now also C11.1, C12.1, C13.1, C14.1, LED1.1 (K)
- net NRST: now also D1.1 (K); no longer C23.2, U1.8 (NRST)
- net VDDA: now also U1.13 (VREF+)
- net VFBSMPS: now also L4.1; no longer L4.2
- net VLXSMPS: now also L4.2; no longer L4.1
- net VBAT: now reaches U1.1 (VBAT)
- net S0: now reaches U1.18 (PA3)
- net S1: now reaches U1.19 (PA4)
- net S2: now reaches U1.20 (PA5)
- net USART_RX: now reaches U1.24 (PA9)
- net USART_TX: now reaches U1.51 (PA10)
- net USER_LED: now reaches U1.65 (PB5)
- net USER_LED: now also LED2.1 (K)
- net VDD renamed +3.3V
- net +3.3V: now also C11.2, C12.2, C13.2, C14.2, R11.1, R12.1
- new net: LED1.2 (A), R11.2
- new net: C23.2, D1.2 (A), U1.8 (NRST)
- new net: LED2.2 (A), R12.2
- no-connect marks 1 -> 37
Other:
- note added: "Inspired by:"
- note added: "MCU POWER SUPPLY"
- note added: "POWER & USER LEDs"
- note added: "Subir codigo mediante USART o ST-LINK?"
- moved on the sheet: C15, C16, C17, C18, C19, C20, C21, C22, C23, L3, L4, Y1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

Commit message: updates
Parts:
- added SW1: SW_Push, Button_Switch_SMD:SW_SPST_TL3342, symbol Switch:SW_Push
- C23: value 100uF -> 100nF
Connections:
- net GND: now also SW1.1
- net NRST: now also SW1.2
- net USART_RX: now also U1.66 (PB6); no longer U1.24 (PA9)
- net USART_TX: now also U1.67 (PB7); no longer U1.51 (PA10)
- net DFR0198: now reaches U1.17 (PA2)
- net SEN0308: now reaches U1.23 (PA8)
- net RF1: now reaches U1.31 (RF1)
- net VBAT renamed VBATT
- no-connect marks 37 -> 36
Other:
- note added: "Cambiar I2C pines a PB13 y PB14?"
- note removed: "Subir codigo mediante USART o ST-LINK?"
- moved on the sheet: C23, D1, R10, U1

Commit message: PCB casi lista
Parts:
- removed C11: 100uF, symbol Device:C
- removed CN1: Conn_ARM_JTAG_SWD_10, Connector_PinHeader_1.27mm:PinHeader_2x05_P1.27mm_Vertical, symbol Connector:Conn_ARM_JTAG_SWD_10
- removed D1: BAT54J, Diode_SMD:D_SOD-323F, symbol Diode:BAT54J
- added C10, C21: 100nF, Capacitor_SMD:C_0402_1005Metric, symbol Device:C
- added C20: 100pF, Capacitor_SMD:C_0402_1005Metric, symbol Device:C
- added D1: D_Schottky, Diode_SMD:D_SOD-323, symbol Device:D_Schottky
- added L4: 10nH, Inductor_SMD:L_0402_1005Metric, symbol Device:L
- added R14, R15, R19: 10k, Resistor_SMD:R_0402_1005Metric, symbol Device:R
- added U4: MB85RS256B, Package_SO:SOIC-8_3.9x4.9mm_P1.27mm, symbol Memory_NVRAM:MB85RS256B
- C12, C13, C14, C16, C17, C18, C19: value 100uF -> 100nF; footprint (none) -> Capacitor_SMD:C_0402_1005Metric; Component (none) -> CL05B104KO5NNNC; Manufacturer (none) -> Samsung; Package (none) -> 0402; Supplier (none) -> JLCPCB; Supplier Part # (none) -> C1525; Supplier Part Type (none) -> Basic
- C15: footprint (none) -> Capacitor_SMD:C_0402_1005Metric; Component (none) -> CL05A475MP5NRNC; Manufacturer (none) -> Samsung; Package (none) -> 0402; Supplier (none) -> JLCPCB; Supplier Part # (none) -> C23733; Supplier Part Type (none) -> Basic
- C22: renamed from C20; footprint (none) -> Capacitor_SMD:C_0402_1005Metric; Component (none) -> CL05A475MP5NRNC; Manufacturer (none) -> Samsung; Package (none) -> 0402; Supplier (none) -> JLCPCB; Supplier Part # (none) -> C23733; Supplier Part Type (none) -> Basic
- C23: footprint (none) -> Capacitor_SMD:C_0402_1005Metric; Component (none) -> CL05B104KO5NNNC; Manufacturer (none) -> Samsung; Package (none) -> 0402; Supplier (none) -> JLCPCB; Supplier Part # (none) -> C1525; Supplier Part Type (none) -> Basic
- C24: renamed from C21; value 10pF -> 15pF; footprint (none) -> Capacitor_SMD:C_0402_1005Metric; Component (none) -> 0402CG150J500NT; Manufacturer (none) -> FH; Package (none) -> 0402; Supplier (none) -> JLCPCB; Supplier Part # (none) -> C1548; Supplier Part Type (none) -> Basic
- C25: renamed from C22; value 10pF -> 15pF; footprint (none) -> Capacitor_SMD:C_0402_1005Metric; Component (none) -> 0402CG150J500NT; Manufacturer (none) -> FH; Package (none) -> 0402; Supplier (none) -> JLCPCB; Supplier Part # (none) -> C1548; Supplier Part Type (none) -> Basic
- L3: value 600 -> 600@100MHz; Component FCM1608KF-601T02 -> GZ1608D601TF; Manufacturer TAI-TECH -> Sunlord; Package L_0603 -> 0603; Supplier Part # C127281 -> C1002; Supplier Part Type (none) -> Basic
- L5: renamed from L4; footprint (none) -> Inductor_SMD:L_0805_2012Metric; Component (none) -> SDFL2012S100KTF; Manufacturer (none) -> Sunlord; Package (none) -> 0805; Supplier (none) -> JLCPCB; Supplier Part # (none) -> C1046; Supplier Part Type (none) -> Basic
- LED1: value GREEN -> Green; footprint LED_SMD:LED_0603_1608Metric -> LED_SMD:LED_0805_2012Metric; Component APTD2012LCGCK -> KT-0805G; Manufacturer Kingbright -> Hubei KENTO Elec; Package LED_0805 -> 0805; Supplier Part # C5366381 -> C2297; Supplier Part Type (none) -> Basic
- LED2: value BLUE -> White; footprint LED_SMD:LED_0603_1608Metric -> LED_SMD:LED_0805_2012Metric; Component APTD2012LQBC/D -> KT-0805W; Manufacturer Kingbright -> Hubei KENTO Elec; Package LED_0805 -> 0805; Supplier Part # C5879058 -> C34499; Supplier Part Type (none) -> Basic
- R13: renamed from R10; footprint (none) -> Resistor_SMD:R_0402_1005Metric; Component (none) -> 0402WGF1002TCE; Manufacturer (none) -> UNI-ROYAL; Package (none) -> 0402; Supplier (none) -> JLCPCB; Supplier Part # (none) -> C25744; Supplier Part Type (none) -> Basic
- R16: renamed from R11; value 1k -> 470; footprint (none) -> Resistor_SMD:R_0402_1005Metric; Component (none) -> 0603WAF4700T5E; Manufacturer (none) -> UNI-ROYAL; Package (none) -> 0603; Supplier (none) -> JLCPCB; Supplier Part # (none) -> C23179; Supplier Part Type (none) -> Basic
- R17: renamed from R12; value 1k -> 300; footprint (none) -> Resistor_SMD:R_0402_1005Metric; Component (none) -> 0603WAF3000T5E; Manufacturer (none) -> UNI-ROYAL; Package (none) -> 0603; Supplier (none) -> JLCPCB; Supplier Part # (none) -> C23025; Supplier Part Type (none) -> Basic
- SW1: value SW_Push -> SW_Reset; Component 4*4*1.7 Surface Mount -> TS-1187A-B-A-B; Manufacturer BOOMELE (Boom Precision Elec) -> XKB Connection; Package SMD-4P 5.2x5.2mm -> SMD-4P 5.1x5.1mm; Supplier Part # C10852 -> C318884; Supplier Part Type (none) -> Basic
- U1: Manufacturer STMicroelectronics -> STMicroelectronics; Supplier Part Type (none) -> Extended
- X1: renamed from Y1; Component NX2016SA-32M-EXS00A-CS06465 -> NX2016SA-32M-EXS00A-CS06465; Supplier Part Type (none) -> Extended
- X2: renamed from Y2; Supplier Part Type (none) -> Extended
Connections:
- net +3.3V: now also C10.1, C20.2, R14.2, R15.2, R19.2, U4.8 (VDD); no longer R17.1
- net DFR0198: now also U1.22 (PA7); no longer U1.17 (PA2)
- net GND: now also LED2.1 (K), C10.2, C20.1, C21.1, U4.4 (GND)
- net NRST: now also D1.1 (K)
- net SCL: now also U1.9 (PC0), R14.1; no longer U1.6 (PB8)
- net SDA: now also U1.10 (PC1), R15.1; no longer U1.7 (PB9)
- net USER_LED: now also R17.1, U1.51 (PA10); no longer LED2.1 (K), U1.65 (PB5)
- net VLXSMPS: now also L4.2; no longer L5.2
- net at C23.2, U1.8 (NRST): now also D1.2 (A)
- net GATE_SENS: now reaches U1.11 (PC2)
- net PV_INA: now reaches U1.15 (PA0)
- net CRI_INA: now reaches U1.16 (PA1)
- net SCK: now reaches U1.47 (PB13)
- net SCK: now also U4.6 (SCK)
- net MISO: now reaches U1.48 (PB14)
- net MISO: now also U4.2 (SO)
- net MOSI: now reaches U1.49 (PB15)
- net MOSI: now also U4.5 (SI)
- net CS_FRAM: now reaches U1.52 (PA11)
- net CS_FRAM: now also U4.1 (~{CS})
- net WP_FRAM: now reaches U1.60 (PC12)
- net WP_FRAM: now also U4.3 (~{WP})
- net OSC32_IN renamed LSE_IN
- net OSC32_OUT renamed LSE_OUT
- net OSC_IN renamed HSE_IN
- net OSC_OUT renamed HSE_OUT
- net S0 renamed S0_AEM
- net S1 renamed S1_AEM
- net S2 renamed S2_AEM
- net VBATT renamed VBAT_BACKUP
- net VBAT_BACKUP: now also C21.2
- new net: L4.1, L5.2
- new net: R19.1, U4.7 (~{HOLD})
- new net WAR_INA: U1.17 (PA2)
- no-connect marks 36 -> 24
Other:
- note added: "FRAM"
- note added: "POWER LED"
- note added: "USER LED"
- note removed: "Cambiar I2C pines a PB13 y PB14?"
- note removed: "STLINK"
- moved on the sheet: C12, C13, C14, C15, C16, C17, C18, C19, C22, C24, C25, L3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

Commit message: retoques
Parts:
- C24, C25: value 15pF -> 12pF; Component 0402CG150J500NT -> 0402CG120J500NT; Supplier Part # C1548 -> C1547
- X1: Component NX2016SA-32M-EXS00A-CS06465 -> Q22FA12800025; Manufacturer NDK -> Seiko Epson; Supplier Part # C1986260 -> C187794
Other:
- moved on the sheet: R13
Changed lines of the file:
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@@
 		)
 	)
-	(text_box "		C24*C25\n9 - 2 = ------ ; C24=C25=14pF\n		C24+C25"
+	(text_box "		C24*C25\n9 - 3 = ------ ; C24=C25=12pF\n		C24+C25"
 		(exclude_from_sim no)
 		(at 228.6 85.09 0)
@@
 	(wire
 		(pts
-			(xy 66.04 111.76) (xy 77.47 111.76)
+			(xy 66.04 113.03) (xy 66.04 111.76)
 		)
 		(stroke
@@
 	(wire
 		(pts
+			(xy 66.04 111.76) (xy 77.47 111.76)
+		)
+		(stroke
+			(width 0)
+			(type default)
+		)
+	)
+	(wire
+		(pts
 			(xy 67.31 96.52) (xy 77.47 96.52)
 		)
@@
 	(wire
 		(pts
-			(xy 123.19 160.02) (xy 128.27 160.02)
+			(xy 123.19 160.02) (xy 127 160.02)
 		)
 		(stroke
@@
 	(wire
 		(pts
-			(xy 209.55 146.05) (xy 213.36 146.05)
+			(xy 209.55 146.05) (xy 214.63 146.05)
 		)
 		(stroke
@@
 	(wire
 		(pts
-			(xy 209.55 143.51) (xy 214.63 143.51)
+			(xy 209.55 143.51) (xy 213.36 143.51)
 		)
 		(stroke
@@
 	)
 	(global_label "MISO"
-		(shape input)
-		(at 213.36 146.05 0)
+		(shape output)
+		(at 214.63 146.05 0)
 		(fields_autoplaced yes)
 		(effects
@@
 		)
 		(property "Intersheetrefs" "${INTERSHEET_REFS}"
-			(at 220.9414 146.05 0)
+			(at 222.2114 146.05 0)
 			(effects
 				(font
@@
 	)
 	(global_label "MOSI"
-		(shape output)
-		(at 214.63 143.51 0)
+		(shape input)
+		(at 213.36 143.51 0)
 		(fields_autoplaced yes)
 		(effects
@@
 		)
 		(property "Intersheetrefs" "${INTERSHEET_REFS}"
-			(at 222.2114 143.51 0)
+			(at 220.9414 143.51 0)
 			(effects
 				(font
@@
 	)
 	(global_label "MISO"
-		(shape output)
-		(at 128.27 160.02 0)
+		(shape input)
+		(at 127 160.02 0)
 		(fields_autoplaced yes)
 		(effects
@@
 		)
 		(property "Intersheetrefs" "${INTERSHEET_REFS}"
-			(at 135.8514 160.02 0)
+			(at 134.5814 160.02 0)
 			(effects
 				(font
@@
 	(symbol
 		(lib_id "Device:R")
-		(at 66.04 115.57 180)
+		(at 66.04 116.84 180)
 		(unit 1)
 		(exclude_from_sim no)
@@
 		(fields_autoplaced yes)
 		(property "Reference" "R13"
-			(at 68.58 114.2999 0)
+			(at 68.58 115.5699 0)
 			(effects
 				(font
@@
 		)
 		(property "Value" "10k"
-			(at 68.58 116.8399 0)
+			(at 68.58 118.1099 0)
 			(effects
 				(font
@@
 		)
 		(property "Footprint" "Resistor_SMD:R_0402_1005Metric"
-			(at 67.818 115.57 90)
+			(at 67.818 116.84 90)
 			(effects
 				(font
@@
 		)
 		(property "Datasheet" "~"
-			(at 66.04 115.57 0)
+			(at 66.04 116.84 0)
 			(effects
 				(font
@@
 		)
 		(property "Description" "10kΩ 50V 62.5mW Thick Film Resistor ±1% ±100ppm/℃ 0402 SMD"
-			(at 66.04 115.57 0)
+			(at 66.04 116.84 0)
 			(effects
 				(font
@@
 		)
 		(property "Component" "0402WGF1002TCE"
-			(at 66.04 115.57 0)
+			(at 66.04 116.84 0)
 			(effects
 				(font
@@
 		)
 		(property "Package" "0402"
-			(at 66.04 115.57 0)
+			(at 66.04 116.84 0)
 			(effects
 				(font
@@
 		)
 		(property "Manufacturer" "UNI-ROYAL"
-			(at 66.04 115.57 0)
+			(at 66.04 116.84 0)
 			(effects
 				(font
@@
 		)
 		(property "Supplier Part #" "C25744"
-			(at 66.04 115.57 0)
+			(at 66.04 116.84 0)
 			(effects
 				(font
@@
 		)
 		(property "Supplier" "JLCPCB"
-			(at 66.04 115.57 0)
+			(at 66.04 116.84 0)
 			(effects
 				(font
@@
 		)
 		(property "Supplier Part Type" "Basic"
-			(at 66.04 115.57 0)
+			(at 66.04 116.84 0)
 			(effects
 				(font
@@
 			)
 		)
-		(property "Value" "15pF"
+		(property "Value" "12pF"
 			(at 256.54 72.3899 0)
 			(effects
@@
 			)
 		)
-		(property "Description" "15pF 50V C0G ±5% 0402 Multilayer Ceramic Capacitor SMD"
+		(property "Description" "12pF 50V C0G ±5% 0402 Multilayer Ceramic Capacitor SMD"
 			(at 252.73 71.12 0)
 			(effects
@@
 			)
 		)
-		(property "Supplier Part #" "C1548"
+		(property "Supplier Part #" "C1547"
 			(at 252.73 71.12 0)
 			(effects
@@
 			)
 		)
-		(property "Component" "0402CG150J500NT"
+		(property "Component" "0402CG120J500NT"
 			(at 252.73 71.12 0)
 			(effects
@@
 			)
 		)
-		(property "Value" "15pF"
+		(property "Value" "12pF"
 			(at 236.22 72.3899 0)
 			(effects
@@
 			)
 		)
-		(property "Description" "15pF 50V C0G ±5% 0402 Multilayer Ceramic Capacitor SMD"
+		(property "Description" "12pF 50V C0G ±5% 0402 Multilayer Ceramic Capacitor SMD"
 			(at 232.41 71.12 0)
 			(effects
@@
 			)
 		)
-		(property "Supplier Part #" "C1548"
+		(property "Supplier Part #" "C1547"
 			(at 232.41 71.12 0)
 			(effects
@@
 			)
 		)
-		(property "Component" "0402CG150J500NT"
+		(property "Component" "0402CG120J500NT"
 			(at 232.41 71.12 0)
 			(effects
@@
 	(symbol
 		(lib_id "power:GND")
-		(at 66.04 119.38 0)
+		(at 66.04 120.65 0)
 		(unit 1)
 		(exclude_from_sim no)
@@
 		(fields_autoplaced yes)
 		(property "Reference" "#PWR037"
-			(at 66.04 125.73 0)
+			(at 66.04 127 0)
 			(effects
 				(font
@@
 		)
 		(property "Value" "GND"
-			(at 66.04 124.46 0)
+			(at 66.04 125.73 0)
 			(effects
 				(font
@@
 		)
 		(property "Footprint" ""
-			(at 66.04 119.38 0)
+			(at 66.04 120.65 0)
 			(effects
 				(font
@@
 		)
 		(property "Datasheet" ""
-			(at 66.04 119.38 0)
+			(at 66.04 120.65 0)
 			(effects
 				(font
@@
 		)
 		(property "Description" "Power symbol creates a global label with name \"GND\" , ground"
-			(at 66.04 119.38 0)
+			(at 66.04 120.65 0)
 			(effects
 				(font
@@
 			)
 		)
-		(property "Description" "10pF 32MHz 60Ω SMD2016-4P Crystal"
+		(property "Description" "8pF 32MHz 60Ω SMD2016-4P Crystal"
 			(at 196.85 69.85 0)
 			(effects
@@
 			)
 		)
-		(property "Component" "NX2016SA-32M-EXS00A-CS06465"
+		(property "Component" "Q22FA12800025"
 			(at 196.85 69.85 0)
 			(effects
@@
 			)
 		)
-		(property "Manufacturer" "NDK"
+		(property "Manufacturer" "Seiko Epson"
 			(at 196.85 69.85 0)
 			(effects
@@
 			)
 		)
-		(property "Supplier Part #" "C1986260"
+		(property "Supplier Part #" "C187794"
 			(at 196.85 69.85 0)
 			(effects

Commit message: islas cristales
Connections:
- net GATE_SENS: now also U1.21 (PA6); no longer U1.11 (PC2)
- no-connect marks 24 -> 23
Changed lines of the file:
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@@
-	)
-	(no_connect
-		(at 123.19 96.52)
 	)
 	(no_connect
@@
 	(wire
 		(pts
+			(xy 123.19 96.52) (xy 128.27 96.52)
+		)
+		(stroke
+			(width 0)
+			(type default)
+		)
+	)
+	(wire
+		(pts
 			(xy 33.02 31.75) (xy 36.83 31.75)
 		)
@@
 		(pts
 			(xy 59.69 76.2) (xy 59.69 81.28)
-		)
-		(stroke
-			(width 0)
-			(type default)
-		)
-	)
-	(wire
-		(pts
-			(xy 72.39 134.62) (xy 77.47 134.62)
 		)
 		(stroke
@@
 		)
 	)
+	(global_label "GATE_SENS"
+		(shape output)
+		(at 128.27 96.52 0)
+		(fields_autoplaced yes)
+		(effects
+			(font
+				(size 1.27 1.27)
+			)
+			(justify left)
+		)
+		(property "Intersheetrefs" "${INTERSHEET_REFS}"
+			(at 141.5965 96.52 0)
+			(effects
+				(font
+					(size 1.27 1.27)
+				)
+				(justify left)
+				(hide yes)
+			)
+		)
+	)
 	(global_label "WP_FRAM"
 		(shape output)
@@
 				(hide yes)
 			)
-		)
-	)
-	(global_label "GATE_SENS"
-		(shape output)
-		(at 72.39 134.62 180)
-		(fields_autoplaced yes)
-		(effects
-			(font
-				(size 1.27 1.27)
-			)
-			(justify right)
-		)
-		(property "Intersheetrefs" "${INTERSHEET_REFS}"
-			(at 59.0635 134.62 0)
-			(effects
-				(font
-					(size 1.27 1.27)
-				)
-				(justify right)
-				(hide yes)
-			)

Commit message: pcb sent to jlcpcb
Parts:
- L4: Component LQP15MN10NG02D -> SDCL1005C10NJTDF; Manufacturer Murata Electronics -> Sunlord; Supplier Part # C162639 -> C27147
- R16, R17: footprint Resistor_SMD:R_0402_1005Metric -> Resistor_SMD:R_0603_1608Metric
Changed lines of the file:
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@@
 			)
 		)
-		(property "Footprint" "Resistor_SMD:R_0402_1005Metric"
+		(property "Footprint" "Resistor_SMD:R_0603_1608Metric"
 			(at 256.032 115.57 90)
 			(effects
@@
 			)
 		)
-		(property "Footprint" "Resistor_SMD:R_0402_1005Metric"
+		(property "Footprint" "Resistor_SMD:R_0603_1608Metric"
 			(at 239.522 115.57 90)
 			(effects
@@
 			)
 		)
-		(property "Description" "10nH 1.3Ω 100mA Inductor ±2% 0402 SMD"
+		(property "Description" "10nH 400mΩ 300mA Inductor ±5% 0402 SMD"
 			(at 53.34 90.17 0)
 			(effects
@@
 			)
 		)
-		(property "Manufacturer" " Murata Electronics"
+		(property "Manufacturer" "Sunlord"
 			(at 53.34 90.17 0)
 			(effects
@@
 			)
 		)
-		(property "Supplier Part #" "C162639"
+		(property "Supplier Part #" "C27147"
 			(at 53.34 90.17 0)
 			(effects
@@
 			)
 		)
-		(property "Component" "LQP15MN10NG02D"
+		(property "Component" "SDCL1005C10NJTDF"
 			(at 53.34 90.17 0)
 			(effects
